File: KiCAD/mainboard/_autosave-mainboard.kicad_pcb (KiCad board)
At the start: 2 copper layers, 4 parts, among them IC1 DLPC1438ZEZ, IC2 DLPA2005ERSLT, J1 AXT550124

Commit message: pain! dmd interface grind part 1
Parts:
- turned J1 to 0 degrees
