File: KiCAD/mainboard/DLPA2005_Interface.kicad_sch (KiCad schematic)
At the start: 1 part, among them IC2 DLPA2005ERSLT

Commit message: some doofus goofus
Other:
- note added: "Vallerie"
Changed lines of the file:
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@@
 	(generator_version "9.0")
 	(paper "A4")
+	(text "Vallerie"
+		(exclude_from_sim no)
+		(at 21.844 16.256 0)
+		(effects
+			(font
+				(size 2.286 2.286)
+			)
+		)
+	)
 	(symbol
 		(lib_id "tp_library:DLPA2005ERSLT")

Commit message: Val's edit
Parts:
- added C22: 22u, Capacitor_SMD:C_0603_1608Metric, symbol Device:C
Connections:
- net RESETZ: now reaches IC2.4 (RESETZ)
- no-connect marks 0 -> 2
Changed lines of the file:
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@@
+		)
+	)
+	(no_connect
+		(at 189.23 111.76)
+	)
+	(no_connect
+		(at 170.18 40.64)
+	)
+	(wire
+		(pts
+			(xy 153.67 26.67) (xy 153.67 33.02)
+		)
+		(stroke
+			(width 0)
+			(type default)
+		)
+	)
+	(wire
+		(pts
+			(xy 154.94 26.67) (xy 153.67 26.67)
+		)
+		(stroke
+			(width 0)
+			(type default)
+		)
+	)
+	(hierarchical_label "RESETZ"
+		(shape input)
+		(at 154.94 26.67 0)
+		(effects
+			(font
+				(size 1.27 1.27)
+			)
+			(justify left)
 		)
 	)
@@
 					(unit 1)
 				)
+			)
+		)
+	)
+	(symbol
+		(lib_id "Device:C")
+		(at 190.5 95.25 0)
+		(unit 1)
+		(exclude_from_sim no)
+		(in_bom yes)
+		(on_board yes)
+		(dnp no)
+		(fields_autoplaced yes)
+		(property "Reference" "C22"
+			(at 194.31 93.9799 0)
+			(effects
+				(font
+					(size 1.27 1.27)
+				)
+				(justify left)
+			)
+		)
+		(property "Value" "22u"
+			(at 194.31 96.5199 0)
+			(effects
+				(font
+					(size 1.27 1.27)
+				)
+				(justify left)
+			)
+		)
+		(property "Footprint" "Capacitor_SMD:C_0603_1608Metric"
+			(at 191.4652 99.06 0)
+			(effects
+				(font
+					(size 1.27 1.27)
+				)
+				(hide yes)
+			)
+		)
+		(property "Datasheet" "~"
+			(at 190.5 95.25 0)
+			(effects
+				(font
+					(size 1.27 1.27)
+				)
+				(hide yes)
+			)
+		)
+		(property "Description" "Unpolarized capacitor"
+			(at 190.5 95.25 0)
+			(effects
+				(font
+					(size 1.27 1.27)
+				)
+				(hide yes)
+			)
+		)
+		(property "Part Number" "810-C1608X5R1A226M "
+			(at 190.5 95.25 0)
+			(effects
+				(font
+					(size 1.27 1.27)
+				)
+				(hide yes)
+			)
+		)
+		(pin "1"
+		)
+		(pin "2"
+		)
+		(instances
+			(project ""
+				(path "/38e83f42-2cf9-4799-a46f-ca415d95b90a/9cd29d54-68c1-4b23-aec1-57d737e6ea74"
+					(reference "C22")
+					(unit 1)
+				)
