File: KiCAD/mainboard/DLPA2005_Interface.kicad_sch (KiCad schematic)
At the start: 8 parts, among them IC2 DLPA2005ERSLT

Commit message: added footprints
Parts:
- renumbered C3 to C?, C2 to C?, C1 to C?, R38 to R?, TP1 to TP?, TP2 to TP?
Changed lines of the file:
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@@
 		(dnp no)
 		(fields_autoplaced yes)
-		(property "Reference" "IC?"
+		(property "Reference" "IC2"
 			(at 81.28 46.9198 0)
 			(effects
@@
 		(dnp no)
 		(fields_autoplaced yes)
-		(property "Reference" "C3"
+		(property "Reference" "C?"
 			(at 213.36 73.6599 0)
 			(effects
@@
 		)
 		(instances
+			(project "mainboard"
+				(path "/38e83f42-2cf9-4799-a46f-ca415d95b90a/9cd29d54-68c1-4b23-aec1-57d737e6ea74"
+					(reference "C?")
+					(unit 1)
+				)
+			)
 			(project "DLPA2005_Interface"
 				(path "/6f8e3acb-36fa-4f2a-bfcd-8820be99bbd1"
@@
 		(dnp no)
 		(fields_autoplaced yes)
-		(property "Reference" "C2"
+		(property "Reference" "C?"
 			(at 193.04 73.6599 0)
 			(effects
@@
 		)
 		(instances
+			(project "mainboard"
+				(path "/38e83f42-2cf9-4799-a46f-ca415d95b90a/9cd29d54-68c1-4b23-aec1-57d737e6ea74"
+					(reference "C?")
+					(unit 1)
+				)
+			)
 			(project "DLPA2005_Interface"
 				(path "/6f8e3acb-36fa-4f2a-bfcd-8820be99bbd1"
@@
 		(on_board yes)
 		(dnp no)
-		(property "Reference" "TP1"
+		(property "Reference" "TP?"
 			(at 115.824 25.908 0)
 			(effects
@@
 		)
 		(instances
+			(project "mainboard"
+				(path "/38e83f42-2cf9-4799-a46f-ca415d95b90a/9cd29d54-68c1-4b23-aec1-57d737e6ea74"
+					(reference "TP?")
+					(unit 1)
+				)
+			)
 			(project ""
 				(path "/6f8e3acb-36fa-4f2a-bfcd-8820be99bbd1"
@@
 		(dnp no)
 		(fields_autoplaced yes)
-		(property "Reference" "C1"
+		(property "Reference" "C?"
 			(at 203.2 73.6599 0)
 			(effects
@@
 		)
 		(instances
+			(project "mainboard"
+				(path "/38e83f42-2cf9-4799-a46f-ca415d95b90a/9cd29d54-68c1-4b23-aec1-57d737e6ea74"
+					(reference "C?")
+					(unit 1)
+				)
+			)
 			(project "DLPA2005_Interface"
 				(path "/6f8e3acb-36fa-4f2a-bfcd-8820be99bbd1"
@@
 		(dnp no)
 		(fields_autoplaced yes)
-		(property "Reference" "C?"
+		(property "Reference" "C22"
 			(at 182.88 73.6599 0)
 			(effects
@@
 		(on_board yes)
 		(dnp no)
-		(property "Reference" "R38"
+		(property "Reference" "R?"
 			(at 87.376 27.94 0)
 			(effects
@@
 		)
 		(instances
+			(project "mainboard"
+				(path "/38e83f42-2cf9-4799-a46f-ca415d95b90a/9cd29d54-68c1-4b23-aec1-57d737e6ea74"
+					(reference "R?")
+					(unit 1)
+				)
+			)
 			(project ""
 				(path "/6f8e3acb-36fa-4f2a-bfcd-8820be99bbd1"
@@
 		(on_board yes)
 		(dnp no)
-		(property "Reference" "TP2"
+		(property "Reference" "TP?"
 			(at 124.714 25.908 0)
 			(effects
@@
 		)
 		(instances
+			(project "mainboard"
+				(path "/38e83f42-2cf9-4799-a46f-ca415d95b90a/9cd29d54-68c1-4b23-aec1-57d737e6ea74"
+					(reference "TP?")
+					(unit 1)
+				)
+			)
 			(project ""
 				(path "/6f8e3acb-36fa-4f2a-bfcd-8820be99bbd1"

Commit message: rawr
Parts:
- removed R?: 30.1, symbol Device:R
- added C196: 10uF, symbol Device:C
- added C197, C198, C20: 220nF, symbol Device:C
- added C199: 2.2uF, symbol Device:C
- added C200, C201: 1uF, symbol Device:C
- added C211, C212, C30, C31: 22uF, Capacitor_SMD:C_0603_1608Metric, symbol Device:C
- added C27, C29: 100nF, symbol Device:C
- added C4, C5, C6: C, symbol Device:C
- added D18: D_Schottky, symbol Device:D_Schottky
- added L1: L, symbol Device:L
- added L2, L3: 2.2uH, symbol Device:L
- added P1P8V, TP22, TP23, TP24, TP3, TP35: TestPoint, symbol Connector:TestPoint
- added R1: R_US, symbol Device:R_US
- added R83: 30.1, symbol Device:R_US
- added R84: 10k, symbol Device:R_US
- added R94: 39m, symbol Device:R_US
- C168, C21, C22: renamed from C?; value 22u -> 22uF
- C169: renamed from C22; value 22u -> 22uF
- gave numbers to parts that had none: 2
Connections:
- net SPI1_MISO: now also R83.1
- net P5V: now reaches IC2.1 (VINL_1)
- net P5V: now also C168.1, C169.1, C21.1, C22.1, IC2.10 (VINR), IC2.18 (VINA), IC2.2 (VINL_2), IC2.25 (VINC), C196.1, C201.1, C27.1, C5.1
- net at IC2.11 (SWN): now also D18.1 (K), L1.2
- net GND: now reaches IC2.12 (PGNDR)
- net GND: now also C168.2, C169.2, C21.2, C22.2, IC2.20 (GND), IC2.23 (PGNDC), IC2.45 (PGNDL_1), IC2.46 (PGNDL_2), IC2.5 (AGND1), C196.2, C197.1, C198.1, C199.2, C20.2, C200.2, C201.2, C211.2, C212.2, C27.2, C29.2, C30.2, C31.2, C4.1, C5.2, C6.2, R1.1, R84.1, R94.2
- net at IC2.13 (SWP): now also L1.1
- net VRST: now reaches IC2.14 (CNTR_VRST)
- net VRST: now also C20.1, D18.2 (A), TP22.1
- net VBIAS: now reaches IC2.15 (VBIAS)
- net VBIAS: now also C197.2, TP24.1
- net VOFS: now reaches IC2.17 (VOFS)
- net VOFS: now also C198.2, TP23.1
- net V2V5: now reaches IC2.19 (V2V5)
- net V2V5: now also C199.1
- net at IC2.21 (LS_OUT): now also C200.1, TP3.1
- net at IC2.22 (LS_IN): now also P1P8V.1
- net at IC2.24 (SWC): now also L3.1
- net RC_CHARGE: now reaches IC2.26 (PWM_IN)
- net P1P1V: now reaches IC2.29 (VCORE)
- net P1P1V: now also C4.2, L3.2, TP35.1
- net at IC2.30 (SENS2): now also TP36.1
- net at IC2.31 (LED_SEL0): now also R1.2
- net P1P8V_DLPC: now reaches IC2.32 (VSPI)
- net P1P8V_DLPC: now also C6.1
- net at IC2.33 (SENS1): now also TP38.1
- net V6V: now reaches IC2.35 (V6V)
- net V6V: now also C29.1
- net at IC2.36 (RLIM_K): now also IC2.40 (RLIM), R94.1
- net at IC2.41 (VLED_1): now also IC2.42 (VLED_2), C211.1, C212.1, C30.1, C31.1
- net at IC2.43 (L2_1): now also IC2.44 (L2_2), L2.1
- net at IC2.47 (L1_1): now also IC2.48 (L1_2), L2.2
- net INTZ: now reaches IC2.6 (INTZ)
- net INTZ: now also R84.2
- net at IC2.9 (SPI_DOUT): now also R83.2
- no-connect marks 0 -> 3
Other:
- note added: "1/4W"
- note added: "CBL2012T100M"
- note added: "Connects to thermal?"
- note added: "DR74-2R2-R"
- note added: "LQM2HPN2R2MG0L"
- note added: "PMEG4002EL,315"
- note added: "What's the R value?"
- note added: "what's EP?"
- moved on the sheet: C168, C169, C21, C22

Commit message: designator names on global finally
Parts:
- renumbered C169 to C22, C21 to C?, C31 to C?, C20 to C?, C30 to C?, C168 to C?, C211 to C?, C199 to C?, C27 to C?, C22 to C?, C201 to C?, C198 to C?, C200 to C?, C212 to C?, C5 to C?, C29 to C?, C4 to C?, C197 to C?, C196 to C?, C6 to C?, D18 to D?, L3 to L?, L2 to L?, L1 to L?, P1P8V to P1P8V?, R1 to R?, R83 to R?, R94 to R?, R84 to R?, TP38 to TP?, TP22 to TP?, TP35 to TP?, TP24 to TP?, TP23 to TP?, TP3 to TP?, TP36 to TP?

Commit message: removed question marks
Connections:
- net GND: now also IC2.49 (EP)
- no-connect marks 3 -> 4
Other:
- note removed: "what's EP?"
Changed lines of the file:
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@@
 		)
 	)
-	(text "what's EP?"
-		(exclude_from_sim no)
-		(at 170.434 134.62 0)
-		(effects
-			(font
-				(size 1.27 1.27)
-			)
-		)
-	)
 	(text "What's the R value?\n"
 		(exclude_from_sim no)
@@
 	)
 	(junction
+		(at 163.83 129.54)
+		(diameter 0)
+		(color 0 0 0 0)
+	)
+	(junction
 		(at 68.58 68.58)
 		(diameter 0)
@@
 	)
 	(junction
+		(at 163.83 119.38)
+		(diameter 0)
+		(color 0 0 0 0)
+	)
+	(junction
 		(at 189.23 43.18)
 		(diameter 0)
@@
 	)
 	(junction
-		(at 168.91 114.3)
+		(at 177.8 73.66)
 		(diameter 0)
 		(color 0 0 0 0)
 	)
 	(junction
-		(at 177.8 73.66)
+		(at 163.83 124.46)
 		(diameter 0)
 		(color 0 0 0 0)
@@
 	)
 	(junction
+		(at 163.83 114.3)
+		(diameter 0)
+		(color 0 0 0 0)
+	)
+	(junction
 		(at 67.31 96.52)
 		(diameter 0)
@@
 		(at 85.09 104.14)
 	)
+	(no_connect
+		(at 3.81 153.67)
+	)
 	(wire
 		(pts
@@
 	(wire
 		(pts
-			(xy 168.91 114.3) (xy 163.83 114.3)
-		)
-		(stroke
-			(width 0)
-			(type default)
-		)
-	)
-	(wire
-		(pts
 			(xy 199.39 73.66) (xy 209.55 73.66)
 		)
@@
 	(wire
 		(pts
-			(xy 163.83 129.54) (xy 171.45 129.54)
-		)
-		(stroke
-			(width 0)
-			(type default)
-		)
-	)
-	(wire
-		(pts
 			(xy 163.83 55.88) (xy 163.83 38.1)
 		)
@@
 	(wire
 		(pts
-			(xy 168.91 111.76) (xy 168.91 114.3)
+			(xy 68.58 57.15) (xy 68.58 53.34)
 		)
 		(stroke
@@
 	(wire
 		(pts
-			(xy 68.58 57.15) (xy 68.58 53.34)
+			(xy 209.55 66.04) (xy 219.71 66.04)
 		)
 		(stroke
@@
 	(wire
 		(pts
-			(xy 209.55 66.04) (xy 219.71 66.04)
+			(xy 93.98 170.18) (xy 115.57 170.18)
 		)
 		(stroke
@@
 	(wire
 		(pts
-			(xy 93.98 170.18) (xy 115.57 170.18)
+			(xy 135.89 160.02) (xy 135.89 157.48)
 		)
 		(stroke
@@
 	(wire
 		(pts
-			(xy 135.89 160.02) (xy 135.89 157.48)
+			(xy 163.83 114.3) (xy 163.83 119.38)
 		)
 		(stroke
@@
 	(wire
 		(pts
-			(xy 163.83 111.76) (xy 168.91 111.76)
-		)
-		(stroke
-			(width 0)
-			(type default)
-		)
-	)
-	(wire
-		(pts
 			(xy 40.64 68.58) (xy 43.18 68.58)
 		)
@@
 	(wire
 		(pts
-			(xy 168.91 114.3) (xy 171.45 114.3)
-		)
-		(stroke
-			(width 0)
-			(type default)
-		)
-	)
-	(wire
-		(pts
 			(xy 110.49 167.64) (xy 93.98 167.64)
 		)
@@
 	(wire
 		(pts
-			(xy 163.83 124.46) (xy 171.45 124.46)
+			(xy 68.58 53.34) (xy 76.2 53.34)
 		)
 		(stroke
@@
 	(wire
 		(pts
-			(xy 68.58 53.34) (xy 76.2 53.34)
+			(xy 163.83 124.46) (xy 163.83 129.54)
 		)
 		(stroke
@@
 	(wire
 		(pts
-			(xy 163.83 119.38) (xy 171.45 119.38)
+			(xy 110.49 27.94) (xy 110.49 33.02)
 		)
 		(stroke
@@
 	(wire
 		(pts
-			(xy 110.49 27.94) (xy 110.49 33.02)
+			(xy 49.53 68.58) (xy 68.58 68.58)
 		)
 		(stroke
@@
 	(wire
 		(pts
-			(xy 49.53 68.58) (xy 68.58 68.58)
+			(xy 163.83 129.54) (xy 171.45 129.54)
 		)
 		(stroke
@@
 	(wire
 		(pts
+			(xy 163.83 129.54) (xy 163.83 134.62)
+		)
+		(stroke
+			(width 0)
+			(type default)
+		)
+	)
+	(wire
+		(pts
 			(xy 85.09 93.98) (xy 78.74 93.98)
 		)
@@
 	(wire
 		(pts
+			(xy 163.83 111.76) (xy 163.83 114.3)
+		)
+		(stroke
+			(width 0)
+			(type default)
+		)
+	)
+	(wire
+		(pts
 			(xy 153.67 27.94) (xy 153.67 33.02)
 		)
@@
 	(wire
 		(pts
+			(xy 163.83 119.38) (xy 163.83 124.46)
+		)
+		(stroke
+			(width 0)
+			(type default)
+		)
+	)
+	(wire
+		(pts
 			(xy 77.47 82.55) (xy 77.47 86.36)
 		)
@@
 			(project ""
 				(path "/6f8e3acb-36fa-4f2a-bfcd-8820be99bbd1"
-					(reference "#PWR011")
+					(reference "C31")
 					(unit 1)
 				)
@@
 	(symbol
 		(lib_id "power:GND")
-		(at 171.45 129.54 90)
+		(at 171.45 129.54 0)
 		(unit 1)
 		(exclude_from_sim no)
@@
 		)
 		(property "Value" "GND"
-			(at 175.26 129.5399 90)
+			(at 171.45 134.62 0)
 			(effects
 				(font
 					(size 1.27 1.27)
 				)
-				(justify right)
 			)
 		)
@@
 			(project ""
 				(path "/6f8e3acb-36fa-4f2a-bfcd-8820be99bbd1"
-					(reference "#PWR010")
+					(reference "#PWR03")
 					(unit 1)
 				)
@@
 			(project ""
 				(path "/6f8e3acb-36fa-4f2a-bfcd-8820be99bbd1"
-					(reference "#PWR012")
+					(reference "C201")
 					(unit 1)
 				)
