File: KiCAD/mainboard/_autosave-DLPC1438_Interface.kicad_sch (KiCad schematic)
At the start: 8 parts

Commit message: some schematic layout power
Parts:
- added C1, C2, C3, C4, C?: 100n, Capacitor_SMD:C_0402_1005Metric, symbol Device:C
Connections:
- net VSS is gone; now on net VCC_INTF: IC?.C4 (VSS_1), IC?.C6 (VSS_2), IC?.C8 (VSS_3), IC?.D10 (VSS_6), IC?.D6 (VSS_4), IC?.D8 (VSS_5), IC?.E13 (VSS_8), IC?.E4 (VSS_7), IC?.F4 (VSS_9), IC?.G10 (VSS_20), IC?.G12 (VSS_21), IC?.G13 (VSS_22), IC?.G4 (VSS_15), IC?.G6 (VSS_16), IC?.G7 (VSS_17), IC?.G8 (VSS_18), IC?.G9 (VSS_19), IC?.H10 (VSS_28), IC?.H12 (VSS_29), IC?.H4 (VSS_23), IC?.H6 (VSS_24), IC?.H7 (VSS_25), IC?.H8 (VSS_26), IC?.H9 (VSS_27), IC?.J13 (VSS_36), IC?.J3 (VSS_30), IC?.K10 (VSS_42), IC?.K12 (VSS_43), IC?.K4 (VSS_37), IC?.K6 (VSS_38), IC?.K7 (VSS_39), IC?.K8 (VSS_40), IC?.K9 (VSS_41), IC?.L3 (VSS_44), IC?.M12 (VSS_48), IC?.M4 (VSS_45), IC?.M5 (VSS_46), IC?.M8 (VSS_47)
- net GND: now also C?.2
- net at IC?.D11 (VCC_FLSH): now also C?.1
- net VCC_INTF: now reaches IC?.M3 (VCC_INTF_1)
- net VCC_INTF: now also IC?.N3 (VCC_INTF_3), IC?.N7 (VCC_INTF_4)
