File: KiCAD/mainboard/_autosave-DLPC1438_Interface.kicad_sch (KiCad schematic)
At the start: 38 parts, among them J2 Conn_01x07_Pin, J31 Conn_01x08_Pin, J7 Conn_01x05_Pin, J9 Conn_01x09_Pin, U1 TXS0102DCU

Commit message: non finished changes
Parts:
- added R1: 56, Resistor_SMD:R_0402_1005Metric, symbol Device:R_US
- added TP3: TestPoint, symbol Connector:TestPoint
Connections:
- net P1P8V_DLPC: now also R1.1, TP3.1
- net DLPC_HOST_IRQ: now reaches IC?.N8 (HOST_IRQ)
- net DLPC_HOST_IRQ: now also R1.2
