File: KiCAD/mainboard/_autosave-DLPA2005_Interface.kicad_sch (KiCad schematic)
At the start: 8 parts, among them IC2 DLPA2005ERSLT

Commit message: #stillonthegrind
Connections:
- net RESETZ is gone; now on an unnamed net: IC2.4 (RESETZ)
- net RC_CHARGE: now reaches IC2.26 (PWM_IN)
- net at IC2.30 (SENS2): now also TP2.1
- net at IC2.33 (SENS1): now also TP1.1
Changed lines of the file:
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@@
 		)
+	)
+	(junction
+		(at 156.21 33.02)
+		(diameter 0)
+		(color 0 0 0 0)
 	)
 	(wire
 		(pts
-			(xy 153.67 26.67) (xy 153.67 33.02)
+			(xy 157.48 33.02) (xy 156.21 33.02)
 		)
 		(stroke
@@
 	(wire
 		(pts
-			(xy 154.94 26.67) (xy 153.67 26.67)
-		)
-		(stroke
-			(width 0)
-			(type default)
-		)
-	)
-	(wire
-		(pts
 			(xy 97.79 27.94) (xy 97.79 33.02)
 		)
@@
 		(pts
 			(xy 95.25 27.94) (xy 95.25 33.02)
+		)
+		(stroke
+			(width 0)
+			(type default)
+		)
+	)
+	(wire
+		(pts
+			(xy 135.89 27.94) (xy 135.89 33.02)
+		)
+		(stroke
+			(width 0)
+			(type default)
+		)
+	)
+	(wire
+		(pts
+			(xy 123.19 30.48) (xy 123.19 33.02)
+		)
+		(stroke
+			(width 0)
+			(type default)
+		)
+	)
+	(wire
+		(pts
+			(xy 156.21 33.02) (xy 153.67 33.02)
+		)
+		(stroke
+			(width 0)
+			(type default)
+		)
+	)
+	(wire
+		(pts
+			(xy 120.65 30.48) (xy 120.65 33.02)
+		)
+		(stroke
+			(width 0)
+			(type default)
+		)
+	)
+	(wire
+		(pts
+			(xy 153.67 25.4) (xy 153.67 26.67)
 		)
 		(stroke
@@
 		)
 	)
-	(hierarchical_label "SPI1_MISO"
-		(shape output)
-		(at 92.71 25.4 90)
+	(hierarchical_label "RC_CHARGE"
+		(shape input)
+		(at 135.89 27.94 90)
 		(effects
 			(font
@@
 		)
 	)
-	(hierarchical_label "RESETZ"
-		(shape input)
-		(at 154.94 26.67 0)
+	(hierarchical_label "SPI1_MISO"
+		(shape output)
+		(at 92.71 25.4 90)
 		(effects
 			(font
