File: KiCAD/mainboard/DLPC1438_Interface.kicad_sch (KiCad schematic)
At the start: 94 parts, among them J10 Conn_01x05_Pin, J2 Conn_01x07_Pin, J29 Conn_01x04_Pin, J3 Conn_02x05_Odd_Even, J31 Conn_01x08_Pin, J4 Conn_01x05_Pin, U12 ECS-2520MV-xxx-xx, U13 MX25L3233FM2, U14 SN74AUP1G06DCKR, U16 DLPC1438ZEZ, U22 TXS0102DCU, U37 TXS0102DCU, U5 SN74AUP1G06DCKR, U7 SN74AUP1G06DCKR

Commit message: nothing to report
Connections:
- net ACT_SYNC: no longer names the net of U16.F15 (GPIO_07)
- no-connect marks 22 -> 23
Changed lines of the file:
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@@
 	)
 	(no_connect
+		(at 361.95 247.65)
+	)
+	(no_connect
 		(at 492.76 158.75)
 	)
@@
 		)
 	)
-	(hierarchical_label "ACT_SYNC"
-		(shape input)
-		(at 361.95 247.65 180)
-		(effects
-			(font
-				(size 1.27 1.27)
-			)
-			(justify right)
-		)
-	)
 	(hierarchical_label "DMD_HS_CLK_N"
 		(shape input)
@@
 			(effects
 				(font
-					(size 1.27 1.27)
-					(italic yes)
-				)
-			)
-		)
-	)
-	(netclass_flag ""
-		(length 2.54)
-		(shape diamond)
-		(at 361.95 247.65 0)
-		(fields_autoplaced yes)
-		(effects
-			(font
-				(size 1.27 1.27)
-			)
-			(justify left bottom)
-		)
-		(property "Netclass" "BGA_Signal"
-			(at 363.1565 245.11 0)
-			(effects
-				(font
-					(size 1.27 1.27)
-				)
-				(justify left)
-			)
-		)
-		(property "Component Class" ""
-			(at 57.15 185.42 0)
-			(effects
-				(font

Commit message: more layout stuff
Parts:
- added D5: SML-LX1206SIC-TR, tp_library:LED_SML-LX1206SIC-TR_LUM-M, symbol ul_SML-LX1206SIC-TR:SML-LX1206SIC-TR
- C108, C112, C114, C115, C120, C121, C125, C126, C127, C128, C129, C130, C131, C132, C133, C134, C138, C139, C140, C141, C142, C143, C144, C145, C155, C156, C157, C170, C171, C238, C239, C7: footprint CAPC2012X70 -> tp_library:CAP_CL05_SAM
Connections:
- net P3P3V: now also D5.2; no longer R5.1
- new net: D5.1, R5.1
Changed lines of the file:
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@@
 	(wire
 		(pts
-			(xy 125.73 220.98) (xy 139.7 220.98)
+			(xy 125.73 220.98) (xy 127 220.98)
 		)
 		(stroke
@@
 	(wire
 		(pts
+			(xy 137.16 220.98) (xy 139.7 220.98)
+		)
+		(stroke
+			(width 0)
+			(type default)
+		)
+	)
+	(wire
+		(pts
 			(xy 417.83 102.87) (xy 431.8 102.87)
 		)
@@
 			)
 		)
-		(property "Footprint" "CAPC2012X70"
+		(property "Footprint" "tp_library:CAP_CL05_SAM"
 			(at 513.08 226.06 0)
 			(effects
@@
 	)
 	(symbol
+		(lib_id "ul_SML-LX1206SIC-TR:SML-LX1206SIC-TR")
+		(at 137.16 220.98 0)
+		(mirror y)
+		(unit 1)
+		(exclude_from_sim no)
+		(in_bom yes)
+		(on_board yes)
+		(dnp no)
+		(property "Reference" "D5"
+			(at 130.81 227.33 0)
+			(effects
+				(font
+					(size 1.524 1.524)
+				)
+			)
+		)
+		(property "Value" "SML-LX1206SIC-TR"
+			(at 130.81 224.79 0)
+			(effects
+				(font
+					(size 1.524 1.524)
+				)
+			)
+		)
+		(property "Footprint" "tp_library:LED_SML-LX1206SIC-TR_LUM-M"
+			(at 137.16 220.98 0)
+			(effects
+				(font
+					(size 1.27 1.27)
+					(italic yes)
+				)
+				(hide yes)
+			)
+		)
+		(property "Datasheet" "SML-LX1206SIC-TR"
+			(at 137.16 220.98 0)
+			(effects
+				(font
+					(size 1.27 1.27)
+					(italic yes)
+				)
+				(hide yes)
+			)
+		)
+		(property "Description" ""
+			(at 137.16 220.98 0)
+			(effects
+				(font
+					(size 1.27 1.27)
+				)
+				(hide yes)
+			)
+		)
+		(pin "2"
+		)
+		(pin "1"
+		)
+		(instances
+			(project "mainboard"
+				(path "/38e83f42-2cf9-4799-a46f-ca415d95b90a/a69a407c-1a7c-4ac9-a9eb-cd67809c5ec0"
+					(reference "D5")
+					(unit 1)
+				)
+			)
+		)
+	)
+	(symbol
 		(lib_id "ERJP06F3301V:ERJP06F3301V")
 		(at 64.77 297.18 90)
@@
 			)
 		)
-		(property "Footprint" "CAPC2012X70"
+		(property "Footprint" "tp_library:CAP_CL05_SAM"
 			(at 251.46 58.42 0)
 			(effects
@@
 			)
 		)
-		(property "Footprint" "CAPC2012X70"
+		(property "Footprint" "tp_library:CAP_CL05_SAM"
 			(at 114.3 228.6 0)
 			(effects
@@
 			)
 		)
-		(property "Footprint" "CAPC2012X70"
+		(property "Footprint" "tp_library:CAP_CL05_SAM"
 			(at 186.69 58.42 0)
 			(effects
@@
 			)
 		)
-		(property "Footprint" "CAPC2012X70"
+		(property "Footprint" "tp_library:CAP_CL05_SAM"
 			(at 260.35 58.42 0)
 			(effects
@@
 			)
 		)
-		(property "Footprint" "CAPC2012X70"
+		(property "Footprint" "tp_library:CAP_CL05_SAM"
 			(at 123.19 133.35 0)
 			(effects
@@
 			)
 		)
-		(property "Footprint" "CAPC2012X70"
+		(property "Footprint" "tp_library:CAP_CL05_SAM"
 			(at 252.73 134.62 0)
 			(effects
@@
 			)
 		)
-		(property "Footprint" "CAPC2012X70"
+		(property "Footprint" "tp_library:CAP_CL05_SAM"
 			(at 58.42 58.42 0)
 			(effects
@@
 			)
 		)
-		(property "Footprint" "CAPC2012X70"
+		(property "Footprint" "tp_library:CAP_CL05_SAM"
 			(at 318.77 132.08 0)
 			(effects
@@
 			)
 		)
-		(property "Footprint" "CAPC2012X70"
+		(property "Footprint" "tp_library:CAP_CL05_SAM"
 			(at 270.51 58.42 0)
 			(effects
@@
 			)
 		)
-		(property "Footprint" "CAPC2012X70"
+		(property "Footprint" "tp_library:CAP_CL05_SAM"
 			(at 242.57 224.79 0)
 			(effects
@@
 			)
 		)
-		(property "Footprint" "CAPC2012X70"
+		(property "Footprint" "tp_library:CAP_CL05_SAM"
 			(at 483.87 180.34 0)
 			(effects
@@
 			)
 		)
-		(property "Footprint" "CAPC2012X70"
+		(property "Footprint" "tp_library:CAP_CL05_SAM"
 			(at 120.65 59.69 0)
 			(effects
@@
 			)
 		)
-		(property "Footprint" "CAPC2012X70"
+		(property "Footprint" "tp_library:CAP_CL05_SAM"
 			(at 72.39 57.15 0)
 			(effects
@@
 			)
 		)
-		(property "Footprint" "CAPC2012X70"
+		(property "Footprint" "tp_library:CAP_CL05_SAM"
 			(at 219.71 58.42 0)
 			(effects
@@
 			)
 		)
-		(property "Footprint" "CAPC2012X70"
+		(property "Footprint" "tp_library:CAP_CL05_SAM"
 			(at 135.89 59.69 0)
 			(effects
@@
 			)
 		)
-		(property "Footprint" "CAPC2012X70"
+		(property "Footprint" "tp_library:CAP_CL05_SAM"
 			(at 210.82 58.42 0)
 			(effects
@@
 			)
 		)
-		(property "Footprint" "CAPC2012X70"
+		(property "Footprint" "tp_library:CAP_CL05_SAM"
 			(at 201.93 58.42 0)
 			(effects
@@
 			)
 		)
-		(property "Footprint" "CAPC2012X70"
+		(property "Footprint" "tp_library:CAP_CL05_SAM"
 			(at 194.31 58.42 0)
 			(effects
@@
 			)
 		)
-		(property "Footprint" "CAPC2012X70"
+		(property "Footprint" "tp_library:CAP_CL05_SAM"
 			(at 66.04 57.15 0)
 			(effects
@@
 			)
 		)
-		(property "Footprint" "CAPC2012X70"
+		(property "Footprint" "tp_library:CAP_CL05_SAM"
 			(at 242.57 134.62 0)
 			(effects
@@
 			)
 		)
-		(property "Footprint" "CAPC2012X70"
+		(property "Footprint" "tp_library:CAP_CL05_SAM"
 			(at 146.05 309.88 0)
 			(effects
@@
 			)
 		)
-		(property "Footprint" "CAPC2012X70"
+		(property "Footprint" "tp_library:CAP_CL05_SAM"
 			(at 95.25 309.88 0)
 			(effects
@@
 			)
 		)
-		(property "Footprint" "CAPC2012X70"
+		(property "Footprint" "tp_library:CAP_CL05_SAM"
 			(at 549.91 139.7 0)
 			(effects
@@
 			)
 		)
-		(property "Footprint" "CAPC2012X70"
+		(property "Footprint" "tp_library:CAP_CL05_SAM"
 			(at 245.11 58.42 0)
 			(effects
@@
 			)
 		)
-		(property "Footprint" "CAPC2012X70"
+		(property "Footprint" "tp_library:CAP_CL05_SAM"
 			(at 142.24 59.69 0)
 			(effects
@@
 			)
 		)
-		(property "Footprint" "CAPC2012X70"
+		(property "Footprint" "tp_library:CAP_CL05_SAM"
 			(at 307.34 181.61 0)
 			(effects
@@
 			)
 		)
-		(property "Footprint" "CAPC2012X70"
+		(property "Footprint" "tp_library:CAP_CL05_SAM"
 			(at 236.22 58.42 0)
 			(effects
@@
 			)
 		)
-		(property "Footprint" "CAPC2012X70"
+		(property "Footprint" "tp_library:CAP_CL05_SAM"
 			(at 227.33 58.42 0)
 			(effects
@@
 			)
 		)
-		(property "Footprint" "CAPC2012X70"
+		(property "Footprint" "tp_library:CAP_CL05_SAM"
 			(at 563.88 147.32 0)
 			(effects
@@
 			)
 		)
-		(property "Footprint" "CAPC2012X70"
+		(property "Footprint" "tp_library:CAP_CL05_SAM"
 			(at 80.01 57.15 0)
 			(effects
@@
 			)
 		)
-		(property "Footprint" "CAPC2012X70"
+		(property "Footprint" "tp_library:CAP_CL05_SAM"
 			(at 128.27 59.69 0)
 			(effects

Commit message: more layout
Changed lines of the file:
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@@
 	(wire
 		(pts
+			(xy 434.34 95.25) (xy 417.83 95.25)
+		)
+		(stroke
+			(width 0)
+			(type default)
+		)
+	)
+	(wire
+		(pts
 			(xy 529.59 288.29) (xy 537.21 288.29)
 		)
@@
 	(wire
 		(pts
+			(xy 433.07 140.97) (xy 417.83 140.97)
+		)
+		(stroke
+			(width 0)
+			(type default)
+		)
+	)
+	(wire
+		(pts
 			(xy 132.08 314.96) (xy 129.54 314.96)
 		)
@@
 	(wire
 		(pts
+			(xy 434.34 184.15) (xy 417.83 184.15)
+		)
+		(stroke
+			(width 0)
+			(type default)
+		)
+	)
+	(wire
+		(pts
 			(xy 331.47 115.57) (xy 361.95 115.57)
 		)
@@
 		)
 	)
+	(wire
+		(pts
+			(xy 433.07 125.73) (xy 417.83 125.73)
+		)
+		(stroke
+			(width 0)
+			(type default)
+		)
+	)
 	(polyline
 		(pts
@@
 		)
 	)
+	(wire
+		(pts
+			(xy 434.34 92.71) (xy 417.83 92.71)
+		)
+		(stroke
+			(width 0)
+			(type default)
+		)
+	)
 	(polyline
 		(pts
@@
 	(wire
 		(pts
+			(xy 433.07 148.59) (xy 417.83 148.59)
+		)
+		(stroke
+			(width 0)
+			(type default)
+		)
+	)
+	(wire
+		(pts
 			(xy 260.35 64.008) (xy 260.35 66.04)
 		)
@@
 		)
 	)
+	(wire
+		(pts
+			(xy 433.07 128.27) (xy 417.83 128.27)
+		)
+		(stroke
+			(width 0)
+			(type default)
+		)
+	)
 	(polyline
 		(pts
@@
 	(wire
 		(pts
+			(xy 433.07 146.05) (xy 417.83 146.05)
+		)
+		(stroke
+			(width 0)
+			(type default)
+		)
+	)
+	(wire
+		(pts
 			(xy 354.33 176.53) (xy 361.95 176.53)
 		)
@@
 	(wire
 		(pts
+			(xy 433.07 57.15) (xy 417.83 57.15)
+		)
+		(stroke
+			(width 0)
+			(type default)
+		)
+	)
+	(wire
+		(pts
 			(xy 433.07 234.95) (xy 433.07 232.41)
 		)
@@
 	(wire
 		(pts
+			(xy 433.07 143.51) (xy 417.83 143.51)
+		)
+		(stroke
+			(width 0)
+			(type default)
+		)
+	)
+	(wire
+		(pts
 			(xy 260.35 66.04) (xy 251.46 66.04)
 		)
@@
 	(wire
 		(pts
+			(xy 433.07 54.61) (xy 417.83 54.61)
+		)
+		(stroke
+			(width 0)
+			(type default)
+		)
+	)
+	(wire
+		(pts
+			(xy 434.34 181.61) (xy 417.83 181.61)
+		)
+		(stroke
+			(width 0)
+			(type default)
+		)
+	)
+	(wire
+		(pts
 			(xy 537.21 143.51) (xy 547.37 143.51)
 		)
@@
 	(wire
 		(pts
+			(xy 434.34 179.07) (xy 417.83 179.07)
+		)
+		(stroke
+			(width 0)
+			(type default)
+		)
+	)
+	(wire
+		(pts
 			(xy 227.33 66.04) (xy 219.71 66.04)
 		)
@@
 	(hierarchical_label "PDATA5"
 		(shape input)
-		(at 417.83 146.05 0)
+		(at 433.07 146.05 0)
 		(effects
 			(font
@@
 	(hierarchical_label "GPIO_18"
 		(shape input)
-		(at 417.83 179.07 0)
+		(at 434.34 179.07 0)
 		(effects
 			(font
@@
 	(hierarchical_label "PDATA3"
 		(shape input)
-		(at 417.83 125.73 0)
+		(at 433.07 125.73 0)
 		(effects
 			(font
@@
 	(hierarchical_label "THERM_PWR"
 		(shape input)
-		(at 417.83 57.15 0)
+		(at 433.07 57.15 0)
 		(effects
 			(font
@@
 	(hierarchical_label "GPIO_16"
 		(shape input)
-		(at 417.83 140.97 0)
+		(at 433.07 140.97 0)
 		(effects
 			(font
@@
 	(hierarchical_label "PDATA0"
 		(shape input)
-		(at 417.83 95.25 0)
+		(at 434.34 95.25 0)
 		(effects
 			(font
@@
 	(hierarchical_label "PDATA2"
 		(shape input)
-		(at 417.83 128.27 0)
+		(at 433.07 128.27 0)
 		(effects
 			(font
@@
 	(hierarchical_label "PDATA4"
 		(shape input)
-		(at 417.83 148.59 0)
+		(at 433.07 148.59 0)
 		(effects
 			(font
@@
 	(hierarchical_label "RC_CHARGE"
 		(shape input)
-		(at 417.83 54.61 0)
+		(at 433.07 54.61 0)
 		(effects
 			(font
@@
 	(hierarchical_label "GPIO_19"
 		(shape input)
-		(at 417.83 181.61 0)
+		(at 434.34 181.61 0)
 		(effects
 			(font
@@
 	(hierarchical_label "GPIO_17"
 		(shape input)
-		(at 417.83 143.51 0)
+		(at 433.07 143.51 0)
 		(effects
 			(font
@@
 	(hierarchical_label "PDATA7"
 		(shape input)
-		(at 417.83 184.15 0)
+		(at 434.34 184.15 0)
 		(effects
 			(font
@@
 	(hierarchical_label "PDATA1"
 		(shape input)
-		(at 417.83 92.71 0)
+		(at 434.34 92.71 0)
 		(effects
 			(font

Commit message: updated footprint to new IEEE folder
Parts:
- R172, R173, R18, R43, R74, R75, R76, R77: footprint RESC2012X60N -> tp_library:RESC1005X40N
Changed lines of the file:
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@@
 			)
 		)
-		(property "Footprint" "RESC2012X60N"
+		(property "Footprint" "tp_library:RESC1005X40N"
 			(at 261.62 234.95 0)
 			(effects
@@
 			)
 		)
-		(property "Footprint" "RESC2012X60N"
+		(property "Footprint" "tp_library:RESC1005X40N"
 			(at 85.09 151.13 0)
 			(effects
@@
 			)
 		)
-		(property "Footprint" "RESC2012X60N"
+		(property "Footprint" "tp_library:RESC1005X40N"
 			(at 326.39 198.12 0)
 			(effects
@@
 			)
 		)
-		(property "Footprint" "RESC2012X60N"
+		(property "Footprint" "tp_library:RESC1005X40N"
 			(at 321.31 74.93 0)
 			(effects
@@
 			)
 		)
-		(property "Footprint" "RESC2012X60N"
+		(property "Footprint" "tp_library:RESC1005X40N"
 			(at 342.9 191.77 0)
 			(effects
@@
 			)
 		)
-		(property "Footprint" "RESC2012X60N"
+		(property "Footprint" "tp_library:RESC1005X40N"
 			(at 323.85 81.28 0)
 			(effects
@@
 			)
 		)
-		(property "Footprint" "RESC2012X60N"
+		(property "Footprint" "tp_library:RESC1005X40N"
 			(at 345.44 156.21 0)
 			(effects
@@
 			)
 		)
-		(property "Footprint" "RESC2012X60N"
+		(property "Footprint" "tp_library:RESC1005X40N"
 			(at 320.04 113.03 0)
 			(effects

Commit message: refactor
Parts:
- R172, R173, R18, R43, R74, R75, R76, R77: footprint tp_library:RESC1005X40N -> RESC2012X60N

Commit message: schematic chagnesS
Parts:
- C238, C239: value 100n -> 100nF
- R44, R45: footprint (none) -> Resistor_SMD:R_0201_0603Metric_Pad0.64x0.40mm_HandSolder
- renumbered R8 to R154
Other:
- moved on the sheet: C108, C112, C114, C115, C120, C121, C125, C126, C127, C128, C129, C130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

Commit message: schematic changes
Parts:
- C120, C121, C125, C126, C128, C129, C130, C131, C132, C133, C134, C139, C140, C141, C142, C143, C144, C145, C155, C156, C157, C7: value 100n -> 100nF
Changed lines of the file:
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@@
 			)
 		)
-		(property "Value" "100n"
+		(property "Value" "100nF"
 			(at 212.344 51.562 0)
 			(show_name no)
@@
 			)
 		)
-		(property "Value" "100n"
+		(property "Value" "100nF"
 			(at 203.454 51.562 0)
 			(show_name no)
@@
 			)
 		)
-		(property "Value" "100n"
+		(property "Value" "100nF"
 			(at 133.604 55.372 0)
 			(show_name no)
@@
 			)
 		)
-		(property "Value" "100n"
+		(property "Value" "100nF"
 			(at 77.47 52.324 0)
 			(show_name no)
@@
 			)
 		)
-		(property "Value" "100n"
+		(property "Value" "100nF"
 			(at 55.626 54.102 0)
 			(show_name no)
@@
 			)
 		)
-		(property "Value" "100n"
+		(property "Value" "100nF"
 			(at 272.034 51.562 0)
 			(show_name no)
@@
 			)
 		)
-		(property "Value" "100n"
+		(property "Value" "100nF"
 			(at 228.854 51.562 0)
 			(show_name no)
@@
 			)
 		)
-		(property "Value" "100n"
+		(property "Value" "100nF"
 			(at 244.348 127.508 0)
 			(show_name no)
@@
 			)
 		)
-		(property "Value" "100n"
+		(property "Value" "100nF"
 			(at 125.984 55.372 0)
 			(show_name no)
@@
 			)
 		)
-		(property "Value" "100n"
+		(property "Value" "100nF"
 			(at 261.874 51.562 0)
 			(show_name no)
@@
 			)
 		)
-		(property "Value" "100n"
+		(property "Value" "100nF"
 			(at 254.254 127.762 0)
 			(show_name no)
@@
 			)
 		)
-		(property "Value" "100n"
+		(property "Value" "100nF"
 			(at 246.634 51.562 0)
 			(show_name no)
@@
 			)
 		)
-		(property "Value" "100n"
+		(property "Value" "100nF"
 			(at 118.618 54.864 0)
 			(show_name no)
@@
 			)
 		)
-		(property "Value" "100n"
+		(property "Value" "100nF"
 			(at 237.744 51.562 0)
 			(show_name no)
@@
 			)
 		)
-		(property "Value" "100n"
+		(property "Value" "100nF"
 			(at 195.834 51.562 0)
 			(show_name no)
@@
 			)
 		)
-		(property "Value" "100n"
+		(property "Value" "100nF"
 			(at 63.246 52.578 0)
 			(show_name no)
@@
 			)
 		)
-		(property "Value" "100n"
+		(property "Value" "100nF"
 			(at 236.474 223.266 0)
 			(show_name no)
@@
 			)
 		)
-		(property "Value" "100n"
+		(property "Value" "100nF"
 			(at 221.234 51.562 0)
 			(show_name no)
@@
 			)
 		)
-		(property "Value" "100n"
+		(property "Value" "100nF"
 			(at 188.214 51.562 0)
 			(show_name no)
@@
 			)
 		)
-		(property "Value" "100n"
+		(property "Value" "100nF"
 			(at 69.596 52.832 0)
 			(show_name no)
@@
 			)
 		)
-		(property "Value" "100n"
+		(property "Value" "100nF"
 			(at 254.762 52.578 0)
 			(show_name no)
@@
 			)
 		)
-		(property "Value" "100n"
+		(property "Value" "100nF"
 			(at 139.954 54.356 0)
 			(show_name no)

Commit message: schematic changes - zero DRC errors but I have things to dicuss, and layout footprint work and rearrangment
Parts:
- added U38: TPD2E001DRYR, tp_library:DRY6, symbol TPD2E001DRYR:TPD2E001DRYR
- C120, C121, C125, C126, C128, C129, C130, C131, C132, C133, C134, C139, C140, C141, C142, C143, C144, C145, C155, C156, C157, C238, C239, C7: Manufacturer_Part_Number CL05B104KO5NNNC -> (none)
Connections:
- net EXT_I2CPWR_F: now also U38.6 (IO2); no longer C239.2, R154.2, R155.2, R158.2, U37.6 (OE), U37.7 (VCCB)
- net EXT_SDA: now also U38.3 (IO1)
- net GND: now also U38.4 (GND)
- new net: C239.2, R154.2, R155.2, R158.2, U37.6 (OE), U37.7 (VCCB)
- new net P5V: U38.1 (VCC)
- no-connect marks 23 -> 21
Other:
- note added: "Flash SPI"
- note added: "JTAG"
- moved on the sheet: J3, J31, R163, R165, R171, R174, TP20, TP21, TP7
