File: KiCAD/mainboard/DMD_Interface.kicad_sch (KiCad schematic)
At the start: 21 parts, among them IC3 SN74AUP1G06DCKR, IC4 SN74AUP1G07DCKR, IC5 SN74AUP1G07DCKR, J1 AXT550124, J10 Conn_01x05_Pin, J30 Conn_01x08_Pin

Commit message: more ERC knocked out
Parts:
- removed J10: Conn_01x05_Pin, Connector_PinHeader_2.54mm:PinHeader_1x05_P2.54mm_Vertical, symbol Connector:Conn_01x05_Pin
Changed lines of the file:
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@@
 	(wire
 		(pts
-			(xy 134.62 152.4) (xy 133.35 152.4)
-		)
-		(stroke
-			(width 0)
-			(type default)
-		)
-	)
-	(wire
-		(pts
 			(xy 110.49 41.148) (xy 110.49 44.45)
 		)
@@
 	(wire
 		(pts
-			(xy 134.62 154.94) (xy 133.35 154.94)
-		)
-		(stroke
-			(width 0)
-			(type default)
-		)
-	)
-	(wire
-		(pts
 			(xy 36.83 88.9) (xy 41.91 88.9)
 		)
@@
 	(wire
 		(pts
-			(xy 134.62 160.02) (xy 133.35 160.02)
-		)
-		(stroke
-			(width 0)
-			(type default)
-		)
-	)
-	(wire
-		(pts
 			(xy 110.49 44.45) (xy 120.65 44.45)
 		)
@@
 	(wire
 		(pts
-			(xy 134.62 157.48) (xy 133.35 157.48)
-		)
-		(stroke
-			(width 0)
-			(type default)
-		)
-	)
-	(wire
-		(pts
 			(xy 152.4 101.6) (xy 162.56 101.6)
 		)
@@
 	(wire
 		(pts
-			(xy 134.62 149.86) (xy 118.11 149.86)
-		)
-		(stroke
-			(width 0)
-			(type default)
-		)
-	)
-	(wire
-		(pts
 			(xy 40.64 73.66) (xy 41.91 73.66)
 		)
@@
 		)
 	)
-	(hierarchical_label "SPI1_MOSI"
-		(shape input)
-		(at 133.35 154.94 180)
-		(effects
-			(font
-				(size 1.27 1.27)
-			)
-			(justify right)
-		)
-	)
 	(hierarchical_label "VRST"
 		(shape input)
@@
 		)
 	)
-	(hierarchical_label "SPI1_CLK"
-		(shape input)
-		(at 133.35 160.02 180)
-		(effects
-			(font
-				(size 1.27 1.27)
-			)
-			(justify right)
-		)
-	)
 	(hierarchical_label "DMD_HS_WDATAA_N"
 		(shape input)
@@
 		)
 	)
-	(hierarchical_label "SPI1_CSZ0"
-		(shape input)
-		(at 133.35 157.48 180)
-		(effects
-			(font
-				(size 1.27 1.27)
-			)
-			(justify right)
-		)
-	)
 	(hierarchical_label "PRINT_ACTIVE"
 		(shape input)
@@
 		)
 	)
-	(hierarchical_label "SPI1_MISO"
-		(shape input)
-		(at 133.35 152.4 180)
-		(effects
-			(font
-				(size 1.27 1.27)
-			)
-			(justify right)
-		)
-	)
 	(hierarchical_label "DMD_HS_WDATAE_P"
 		(shape input)
@@
 	)
 	(symbol
-		(lib_id "Connector:Conn_01x05_Pin")
-		(at 139.7 154.94 0)
-		(mirror y)
-		(unit 1)
-		(exclude_from_sim no)
-		(in_bom yes)
-		(on_board yes)
-		(dnp no)
-		(property "Reference" "J10"
-			(at 129.286 145.542 0)
-			(effects
-				(font
-					(size 1.27 1.27)
-				)
-			)
-		)
-		(property "Value" "Conn_01x05_Pin"
-			(at 129.286 148.082 0)
-			(effects
-				(font
-					(size 1.27 1.27)
-				)
-			)
-		)
-		(property "Footprint" "Connector_PinHeader_2.54mm:PinHeader_1x05_P2.54mm_Vertical"
-			(at 139.7 154.94 0)
-			(effects
-				(font
-					(size 1.27 1.27)
-				)
-				(hide yes)
-			)
-		)
-		(property "Datasheet" "~"
-			(at 139.7 154.94 0)
-			(effects
-				(font
-					(size 1.27 1.27)
-				)
-				(hide yes)
-			)
-		)
-		(property "Description" "Generic connector, single row, 01x05, script generated"
-			(at 139.7 154.94 0)
-			(effects
-				(font
-					(size 1.27 1.27)
-				)
-				(hide yes)
-			)
-		)
-		(pin "1"
-		)
-		(pin "2"
-		)
-		(pin "4"
-		)
-		(pin "3"
-		)
-		(pin "5"
-		)
-		(instances
-			(project "mainboard"
-				(path "/38e83f42-2cf9-4799-a46f-ca415d95b90a/2ef4843e-e813-4038-8f91-df837a4944f8"
-					(reference "J10")
-					(unit 1)
-				)
-			)
-		)
-	)
-	(symbol
 		(lib_id "tp_library:SN74AUP1G07DCKR")
 		(at 138.43 104.14 0)
@@
 	)
 	(symbol
+		(lib_id "power:PWR_FLAG")
+		(at 153.67 64.77 180)
+		(unit 1)
+		(exclude_from_sim no)
+		(in_bom yes)
+		(on_board yes)
+		(dnp no)
+		(property "Reference" "#FLG08"
+			(at 153.67 66.675 0)
+			(effects
+				(font
+					(size 1.27 1.27)
+				)
+				(hide yes)
+			)
+		)
+		(property "Value" "PWR_FLAG"
+			(at 152.908 69.596 0)
+			(effects
+				(font
+					(size 1.27 1.27)
+				)
+			)
+		)
+		(property "Footprint" ""
+			(at 153.67 64.77 0)
+			(effects
+				(font
+					(size 1.27 1.27)
+				)
+				(hide yes)
+			)
+		)
+		(property "Datasheet" "~"
+			(at 153.67 64.77 0)
+			(effects
+				(font
+					(size 1.27 1.27)
+				)
+				(hide yes)
+			)
+		)
+		(property "Description" "Special symbol for telling ERC where power comes from"
+			(at 153.67 64.77 0)
+			(effects
+				(font
+					(size 1.27 1.27)
+				)
+				(hide yes)
+			)
+		)
+		(pin "1"
+		)
+		(instances
+			(project "mainboard"
+				(path "/38e83f42-2cf9-4799-a46f-ca415d95b90a/2ef4843e-e813-4038-8f91-df837a4944f8"
+					(reference "#FLG08")
+					(unit 1)
+				)
+			)
+		)
+	)
+	(symbol
 		(lib_id "CC0805KRX7R9BB104:CC0805KRX7R9BB104")
 		(at 78.74 68.58 90)
@@
 					(unit 1)
 				)
-			)
-		)
-	)
-	(symbol
-		(lib_id "power:GND")
-		(at 118.11 149.86 0)
-		(mirror y)
-		(unit 1)
-		(exclude_from_sim no)
-		(in_bom yes)
-		(on_board yes)
-		(dnp no)
-		(fields_autoplaced yes)
-		(property "Reference" "#PWR09"
-			(at 118.11 156.21 0)
-			(effects
-				(font
-					(size 1.27 1.27)
-				)
-				(hide yes)
-			)
-		)
-		(property "Value" "GND"
-			(at 118.11 154.94 0)
-			(effects
-				(font
-					(size 1.27 1.27)
-				)
-			)
-		)
-		(property "Footprint" ""
-			(at 118.11 149.86 0)
-			(effects
-				(font
-					(size 1.27 1.27)
-				)
-				(hide yes)
-			)
-		)
-		(property "Datasheet" ""
-			(at 118.11 149.86 0)
-			(effects
-				(font
-					(size 1.27 1.27)
-				)
-				(hide yes)
-			)
-		)
-		(property "Description" "Power symbol creates a global label with name \"GND\" , ground"
-			(at 118.11 149.86 0)
-			(effects
-				(font
-					(size 1.27 1.27)
-				)
-				(hide yes)
-			)
-		)
-		(pin "1"
-		)
-		(instances
-			(project "mainboard"
-				(path "/38e83f42-2cf9-4799-a46f-ca415d95b90a/2ef4843e-e813-4038-8f91-df837a4944f8"
-					(reference "#PWR09")
-					(unit 1)
-				)

Commit message: more layout stuff
Parts:
- C116, C13, C137, C14, C15: footprint CC0805KRX7R9BB104:CAPC2012X70 -> tp_library:CAP_CL05_SAM
- C122, C123, C124: footprint CC0805KRX7R9BB104:CAPC2012X70 -> tp_library:CAP_CL05_SAM; Manufacturer_Part_Number TMK105BJ104KV -> CL05B104KO5NNNC
Changed lines of the file:
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@@
 			)
 		)
-		(property "Footprint" "CC0805KRX7R9BB104:CAPC2012X70"
+		(property "Footprint" "tp_library:CAP_CL05_SAM"
 			(at 97.79 106.68 0)
 			(effects
@@
 			)
 		)
-		(property "Footprint" "CC0805KRX7R9BB104:CAPC2012X70"
+		(property "Footprint" "tp_library:CAP_CL05_SAM"
 			(at 110.49 35.56 0)
 			(effects
@@
 			)
 		)
-		(property "Manufacturer_Part_Number" "TMK105BJ104KV"
+		(property "Manufacturer_Part_Number" "CL05B104KO5NNNC"
 			(at 110.49 35.56 0)
 			(effects
@@
 			)
 		)
-		(property "Footprint" "CC0805KRX7R9BB104:CAPC2012X70"
+		(property "Footprint" "tp_library:CAP_CL05_SAM"
 			(at 95.25 34.29 0)
 			(effects
@@
 			)
 		)
-		(property "Footprint" "CC0805KRX7R9BB104:CAPC2012X70"
+		(property "Footprint" "tp_library:CAP_CL05_SAM"
 			(at 73.66 33.02 0)
 			(effects
@@
 			)
 		)
-		(property "Footprint" "CC0805KRX7R9BB104:CAPC2012X70"
+		(property "Footprint" "tp_library:CAP_CL05_SAM"
 			(at 78.74 68.58 0)
 			(effects
@@
 			)
 		)
-		(property "Footprint" "CC0805KRX7R9BB104:CAPC2012X70"
+		(property "Footprint" "tp_library:CAP_CL05_SAM"
 			(at 130.81 35.56 0)
 			(effects
@@
 			)
 		)
-		(property "Manufacturer_Part_Number" "TMK105BJ104KV"
+		(property "Manufacturer_Part_Number" "CL05B104KO5NNNC"
 			(at 130.81 35.56 0)
 			(effects
@@
 			)
 		)
-		(property "Footprint" "CC0805KRX7R9BB104:CAPC2012X70"
+		(property "Footprint" "tp_library:CAP_CL05_SAM"
 			(at 83.82 34.29 0)
 			(effects
@@
 			)
 		)
-		(property "Footprint" "CC0805KRX7R9BB104:CAPC2012X70"
+		(property "Footprint" "tp_library:CAP_CL05_SAM"
 			(at 120.65 34.29 0)
 			(effects
@@
 			)
 		)
-		(property "Manufacturer_Part_Number" "TMK105BJ104KV"
+		(property "Manufacturer_Part_Number" "CL05B104KO5NNNC"
 			(at 120.65 34.29 0)
 			(effects

Commit message: refactor
Connections:
- net P3V3V renamed P3P3V

Commit message: schematic chagnesS
Parts:
- removed C137: 100n, tp_library:CAP_CL05_SAM, symbol CC0805KRX7R9BB104:CC0805KRX7R9BB104
- added C60: 100nF, Capacitor_SMD:C_0402_1005Metric_Pad0.74x0.62mm_HandSolder, symbol Device:C
- C122, C123, C124, C13, C14, C15: value 100n -> 100nF
Connections:
- net GND: now also C60.2
- net P1P8V_DLPC: now also C60.1

Commit message: schematic changes
Parts:
- C116: value 100n -> 100nF
Changed lines of the file:
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@@
 			)
 		)
-		(property "Value" "100n"
+		(property "Value" "100nF"
 			(at 85.344 62.992 0)
 			(show_name no)

Commit message: schematic changes - zero DRC errors but I have things to dicuss, and layout footprint work and rearrangment
Parts:
- C116, C122, C123, C124, C13, C14, C15: Manufacturer_Part_Number CL05B104KO5NNNC -> (none)
- C60: footprint Capacitor_SMD:C_0402_1005Metric_Pad0.74x0.62mm_HandSolder -> tp_library:ul_CL05B104KO5NNNC
Changed lines of the file:
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@@
 			)
 		)
-		(property "Datasheet" "TMK105BJ104KV-F"
+		(property "Datasheet" ""
 			(at 100.33 31.75 0)
 			(hide yes)
@@
 			)
 		)
-		(property "Manufacturer_Part_Number" "CL05B104KO5NNNC"
+		(property "Manufacturer_Part_Number" ""
 			(at 100.33 31.75 0)
 			(hide yes)
@@
 			)
 		)
-		(property "Datasheet" "TMK105BJ104KV-F"
+		(property "Datasheet" ""
 			(at 78.74 30.48 0)
 			(hide yes)
@@
 			)
 		)
-		(property "Manufacturer_Part_Number" "CL05B104KO5NNNC"
+		(property "Manufacturer_Part_Number" ""
 			(at 78.74 30.48 0)
 			(hide yes)
@@
 			)
 		)
-		(property "Manufacturer_Part_Number" "CL05B104KO5NNNC"
+		(property "Manufacturer_Part_Number" ""
 			(at 135.89 33.02 0)
 			(hide yes)
@@
 			)
 		)
-		(property "Footprint" "Capacitor_SMD:C_0402_1005Metric_Pad0.74x0.62mm_HandSolder"
+		(property "Footprint" "tp_library:ul_CL05B104KO5NNNC"
 			(at 103.8352 111.76 0)
 			(hide yes)
@@
 			)
 		)
-		(property "Datasheet" "TMK105BJ104KV-F"
+		(property "Datasheet" ""
 			(at 88.9 31.75 0)
 			(hide yes)
@@
 			)
 		)
-		(property "Manufacturer_Part_Number" "CL05B104KO5NNNC"
+		(property "Manufacturer_Part_Number" ""
 			(at 88.9 31.75 0)
 			(hide yes)
@@
 			)
 		)
-		(property "Manufacturer_Part_Number" "CL05B104KO5NNNC"
+		(property "Manufacturer_Part_Number" ""
 			(at 125.73 31.75 0)
 			(hide yes)
@@
 			)
 		)
-		(property "Manufacturer_Part_Number" "CL05B104KO5NNNC"
+		(property "Manufacturer_Part_Number" ""
 			(at 83.82 66.04 0)
 			(hide yes)
@@
 			)
 		)
-		(property "Manufacturer_Part_Number" "CL05B104KO5NNNC"
+		(property "Manufacturer_Part_Number" ""
 			(at 115.57 33.02 0)
 			(hide yes)
