File: KiCAD/mainboard/power_input&generation.kicad_sch (KiCad schematic)
At the start: 51 parts, among them Q1 PMOS, U1 XAL5030-472MEC, U2 LMR33610BDDAR, U26 TPS54340DDA, U3 LMR33610BDDAR, U39 TPS62260DDCT

Commit message: refactor
Parts:
- removed D13: D_Zener, symbol Device:D_Zener
- removed Q1: PMOS, symbol Simulation_SPICE:PMOS
- removed R127: 100k, RES_RMCF0805_STP, symbol RMCF0805FG100K:RMCF0805FG100K
- removed R137: 20k, Resistor_SMD:R_0402_1005Metric, symbol Device:R_US
- removed R138: 15k, Resistor_SMD:R_0402_1005Metric, symbol Device:R_US
- added C111, C113: 100nF, Capacitor_SMD:C_0603_1608Metric_Pad1.08x0.95mm_HandSolder, symbol Device:C
- added IC1: SN74AUP1G06DCKR, tp_library:SOT65P210X110-5N, symbol tp_library:SN74AUP1G06DCKR
- added J5: EJ508B, tp_library:MPD_EJ508B, symbol tp_library:EJ508B
- added R160, R161, R162: 10k, Resistor_SMD:R_0402_1005Metric, symbol Device:R_US
- added SW2: 100SP1T1B4M2QE, tp_library:SW_100SP1T1B4M2QE, symbol tp_library:100SP1T1B4M2QE
- added U6: 74AHC1G08, Package_TO_SOT_SMD:SOT-353_SC-70-5, symbol 74xGxx:74AHC1G08
- added U8: 74AHC1G32, Package_TO_SOT_SMD:SOT-353_SC-70-5, symbol 74xGxx:74AHC1G32
Connections:
- net EXT_VIN: now also C19.1, C25.1, U26.2 (VIN), J5.1
- net FPGA_PWREN: now also U6.4
- net GND: now also C111.2, C113.2, IC1.3 (GND), J5.3, R160.1, R161.2, U6.3 (GND), U8.3 (GND)
- net P3V3V renamed P3P3V_SB
- net P3P3V_SB: now also IC1.5 (VCC), R162.1, U6.5 (VCC), U8.5 (VCC)
- net VIN_LED: no longer names the net of D12.2 (A), R117.1
- new net: R161.1, SW2.1
- new net: R162.2, SW2.3
- new net FE_PROJ_ON: C111.1, R160.2, U8.1
- new net INTZ: U6.2
- new net PROJ_ON: IC1.2 (A), U6.1, U8.4
- new net PROJ_ON_DRV: IC1.4 (Y)
- new net SW_PROJ_ON: C113.1, SW2.2, U8.2
- no-connect marks 2 -> 3
Other:
- note added: "5V to 3V3 Standby Converter (Power Sequencing Intermediary)"
- note added: "EXT Adapter to 5V Converter"
- note removed: "5V to 3V3 Buck Converter"
- note removed: "Adapter to 5V Converter"

Commit message: some extra work
Parts:
- removed C16: 4.7uF, Capacitor_SMD:C_0603_1608Metric_Pad1.08x0.95mm_HandSolder, symbol Device:C
- removed C17: 220nF, Capacitor_SMD:C_0603_1608Metric_Pad1.08x0.95mm_HandSolder, symbol Device:C
- removed C18, C23, C24, C28: 22uF, Capacitor_SMD:C_0603_1608Metric_Pad1.08x0.95mm_HandSolder, symbol Device:C
- removed C32: 100nF, Capacitor_SMD:C_0603_1608Metric_Pad1.08x0.95mm_HandSolder, symbol Device:C
- added C34: 10uF, Capacitor_SMD:C_0603_1608Metric_Pad1.08x0.95mm_HandSolder, symbol Device:C
- added C37, C38, C39: 22uF, Capacitor_SMD:C_0603_1608Metric_Pad1.08x0.95mm_HandSolder, symbol Device:C
- added C40, C45, C49, C55, C58: 100nF, Capacitor_SMD:C_0603_1608Metric_Pad1.08x0.95mm_HandSolder, symbol Device:C
- added C46, C50, C65: 1uF, Capacitor_SMD:C_0603_1608Metric_Pad1.08x0.95mm_HandSolder, symbol Device:C
- added C47, C56: 4.7uF, Capacitor_SMD:C_0603_1608Metric_Pad1.08x0.95mm_HandSolder, symbol Device:C
- added C48, C57: 220nF, Capacitor_SMD:C_0603_1608Metric_Pad1.08x0.95mm_HandSolder, symbol Device:C
- added C54: 53, Capacitor_SMD:C_0603_1608Metric_Pad1.08x0.95mm_HandSolder, symbol Device:C
- added C59: 4.7pF, Capacitor_SMD:C_0603_1608Metric_Pad1.08x0.95mm_HandSolder, symbol Device:C
- added C61: 10pF, Capacitor_SMD:C_0603_1608Metric_Pad1.08x0.95mm_HandSolder, symbol Device:C
- added C64: 18pF, Capacitor_SMD:C_0603_1608Metric_Pad1.08x0.95mm_HandSolder, symbol Device:C
- added D13: LED, LED_SMD:LED_0603_1608Metric_Pad1.05x0.95mm_HandSolder, symbol Device:LED
- added L4, L5: SRU1038-3R5Y, tp_library:IND_BOURNS_SRU1038, symbol tp_library:SRU1038-3R5Y
- added L7: DR1040-5R2-R, tp_library:DR1040, symbol tp_library:DR1040-5R2-R
- added R101, R108, R196, R97: 10k, Resistor_SMD:R_0402_1005Metric, symbol Device:R_US
- added R102: 499k, Resistor_SMD:R_0402_1005Metric, symbol Device:R_US
- added R103, R104, R110: 100k, Resistor_SMD:R_0402_1005Metric, symbol Device:R_US
- added R109: 43.2k, Resistor_SMD:R_0402_1005Metric, symbol Device:R_US
- added R162: 200, Resistor_SMD:R_0402_1005Metric, symbol Device:R_US
- added R98: 124k, Resistor_SMD:R_0402_1005Metric, symbol Device:R_US
- added U4: LMR33610BDDAR, Package_SO:Texas_HSOP-8-1EP_3.9x4.9mm_P1.27mm_ThermalVias, symbol Regulator_Switching:LMR33610BDDAR
- renumbered C8 to C32, C11 to C33, C9 to C34, C10 to C35, C12 to C36
Connections:
- net EXT_VIN: now also C43.1, C44.1, U2.2 (VIN), U3.2 (VIN), C47.1, C48.1, C56.1, C57.1, R196.1, U4.2 (VIN)
- net FPGA_PWREN: now also U4.3 (EN); no longer U3.3 (EN)
- net GND: now also C32.2, C33.2, C34.2, C35.2, C36.2, C34.2, C37.2, C38.2, C39.2, C40.2, C46.2, C47.2, C48.2, C50.2, C54.2, C55.2, C56.2, C57.2, C65.2, R102.2, R109.2, R98.2, U4.1 (GND), U4.9 (GND)
- net P1P2V_BOOT: now also C45.2; no longer U3.7 (BOOT)
- net P1P2V_SW: now also C45.1, L4.2; no longer U3.8 (SW)
- net P3P3V_SB: now also D13.2 (A), R101.2, R108.2, R97.2
- net PROJ_ON_DRV: now also R162.2
- net P1P2V: now reaches C32.1, C33.1, C34.1, C35.1, C36.1
- net P1P2V: now also C59.1, L4.1, R103.1
- net P1P2V_PG: now reaches U2.4 (PG)
- net P1P2V_PG: now also R101.1
- net P1P2V_FB: now reaches U2.5 (FB)
- net P1P2V_FB: now also C59.2, R102.1, R103.2
- net P1P2V_VCC: now reaches U2.6 (VCC)
- net P1P2V_VCC: now also C46.1
- net P1P8V_PG: now reaches U3.4 (PG)
- net P1P8V_PG: now also R97.1
- net P1P8V_FB: now reaches U3.5 (FB)
- net P1P8V_FB: now also C61.2, R104.2, R98.1
- net P1P8V_VCC: now reaches U3.6 (VCC)
- net P1P8V_VCC: now also C50.1
- new net: D13.1 (K), R162.1
- new net P1P8V: C37.1, C38.1, C39.1, C40.1, C61.1, L5.1, R104.1
- new net P1P8V_BOOT: C49.2, U3.7 (BOOT)
- new net P1P8V_EN: R196.2, U3.3 (EN)
- new net P1P8V_SW: C49.1, L5.2, U3.8 (SW)
- new net P3P3V: C34.1, C54.1, C55.1, C64.1, L7.2, R110.1
- new net P3P3V_BOOT: C58.2, U4.7 (BOOT)
- new net P3P3V_FB: C64.2, R109.1, R110.2, U4.5 (FB)
- new net P3P3V_PG: R108.1, U4.4 (PG)
- new net P3P3V_SW: C58.1, L7.1, U4.8 (SW)
- new net P3P3V_VCC: C65.1, U4.6 (VCC)
Other:
- note added: "STBY 3V3 To 1.2V Converter"
- note added: "STBY 3V3 To 1.8V Converter"
- note added: "STBY 3V3 To 3.3V Converter"
- note removed: "3V3 To 1.2V Converter"
- note removed: "3V3 To 1.8V Converter"
- moved on the sheet: C1, C109, C110, C111, C113, C19, C2, C25, C26, C3, C32, C33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

Commit message: schematic chagnesS
Parts:
- removed R161, R162: 10k, Resistor_SMD:R_0402_1005Metric, symbol Device:R_US
- added R214, R216: 10k, Resistor_SMD:R_0402_1005Metric, symbol Device:R_US
- C111, C113, C36, C40, C45, C49, C55, C58: footprint Capacitor_SMD:C_0603_1608Metric_Pad1.08x0.95mm_HandSolder -> Capacitor_SMD:C_0402_1005Metric_Pad0.74x0.62mm_HandSolder; Manufacturer_Name GRM188C81E475KE11D -> CL05B104KO5NNNC
- C32, C33, C34, C35, C37, C38, C39: Manufacturer_Name GRM188C81E475KE11D -> C1608X5R1A226M080AC
- C43, C47, C56: footprint Capacitor_SMD:C_0603_1608Metric_Pad1.08x0.95mm_HandSolder -> Capacitor_SMD:C_0805_2012Metric_Pad1.18x1.45mm_HandSolder
- C44, C48, C57: footprint Capacitor_SMD:C_0603_1608Metric_Pad1.08x0.95mm_HandSolder -> Capacitor_SMD:C_0402_1005Metric_Pad0.74x0.62mm_HandSolder; Manufacturer_Name GRM188C81E475KE11D -> GRM155R6YA224KE01D
- C46, C50: Manufacturer_Name GRM188C81E475KE11D -> CL05A105KA5NQNC
- C53: renamed from C34; footprint Capacitor_SMD:C_0603_1608Metric_Pad1.08x0.95mm_HandSolder -> Capacitor_SMD:C_0805_2012Metric_Pad1.18x1.45mm_HandSolder; Manufacturer_Name GRM188C81E475KE11D -> C2012X5R1V106M085AC
- C54: value 53 -> 10uF; footprint Capacitor_SMD:C_0603_1608Metric_Pad1.08x0.95mm_HandSolder -> Capacitor_SMD:C_0805_2012Metric_Pad1.18x1.45mm_HandSolder; Manufacturer_Name GRM188C81E475KE11D -> C2012X5R1V106M085AC
- C59: footprint Capacitor_SMD:C_0603_1608Metric_Pad1.08x0.95mm_HandSolder -> Capacitor_SMD:C_0402_1005Metric_Pad0.74x0.62mm_HandSolder; Manufacturer_Name GRM188C81E475KE11D -> GCM1555C1H4R7CA16D
- C61: footprint Capacitor_SMD:C_0603_1608Metric_Pad1.08x0.95mm_HandSolder -> Capacitor_SMD:C_0402_1005Metric_Pad0.74x0.62mm_HandSolder; Manufacturer_Name GRM188C81E475KE11D -> KGM05ACG1H100JH
- C64: footprint Capacitor_SMD:C_0603_1608Metric_Pad1.08x0.95mm_HandSolder -> Capacitor_SMD:C_0402_1005Metric_Pad0.74x0.62mm_HandSolder; Manufacturer_Name GRM188C81E475KE11D -> CGA2B2C0G1H180J050BA
- C65: footprint Capacitor_SMD:C_0603_1608Metric_Pad1.08x0.95mm_HandSolder -> Capacitor_SMD:C_0402_1005Metric_Pad0.74x0.62mm_HandSolder; Manufacturer_Name GRM188C81E475KE11D -> CL05A105KA5NQNC
- R102: Manufacturer_Part_Number RC0402FR-0710KL -> MCR01MZPF4993
- R103, R104, R110: Manufacturer_Part_Number RC0402FR-0710KL -> CRCW0402100KFKED
- R109: Manufacturer_Part_Number RC0402FR-0710KL -> RC0402JR-073RL
- R162: Manufacturer_Part_Number RC0402FR-0710KL -> ERJ-2RKF2000X
- R98: Manufacturer_Part_Number RC0402FR-0710KL -> ERJ-2RKF1243X
Connections:
- net GND: now also R214.2
- net P3P3V_SB: now also R216.1
- net at SW2.1: now also R214.1
- net at SW2.3: now also R216.2

Commit message: schematic changes
Changed lines of the file:
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@@
+		)
+	)
+	(label "P1P8V_SW"
+		(at 240.03 71.12 0)
+		(effects
+			(font
+				(size 1.27 1.27)
+			)
+			(justify left bottom)
 		)
 	)
@@
 		)
 	)
+	(label "P1P2V_SW"
+		(at 243.84 30.48 0)
+		(effects
+			(font
+				(size 1.27 1.27)
+			)
+			(justify left bottom)
+		)
+	)
 	(label "P1P2V_VCC"
 		(at 220.98 38.1 180)
@@
 		)
 	)
+	(label "P1P8V_BOOT"
+		(at 240.03 68.58 0)
+		(effects
+			(font
+				(size 1.27 1.27)
+			)
+			(justify left bottom)
+		)
+	)
 	(label "P1P2V_PG"
 		(at 241.3 38.1 0)
@@
 		)
 	)
+	(label "P1P2V_BOOT"
+		(at 243.84 27.94 0)
+		(effects
+			(font
+				(size 1.27 1.27)
+			)
+			(justify left bottom)
+		)
+	)
 	(label "P1P2V_FB"
 		(at 241.3 35.56 0)
@@
 		)
 	)
-	(hierarchical_label "P1P2V_SW"
-		(shape input)
-		(at 243.84 30.48 0)
-		(effects
-			(font
-				(size 1.27 1.27)
-			)
-			(justify left)
-		)
-	)
-	(hierarchical_label "P1P8V_BOOT"
-		(shape input)
-		(at 240.03 68.58 0)
-		(effects
-			(font
-				(size 1.27 1.27)
-			)
-			(justify left)
-		)
-	)
 	(hierarchical_label "P3P3V_SW"
 		(shape input)
@@
 		)
 	)
-	(hierarchical_label "P1P8V_SW"
-		(shape input)
-		(at 240.03 71.12 0)
-		(effects
-			(font
-				(size 1.27 1.27)
-			)
-			(justify left)
-		)
-	)
 	(hierarchical_label "P3P3V_BOOT"
 		(shape input)
@@
 		)
 	)
-	(hierarchical_label "P1P2V_BOOT"
-		(shape input)
-		(at 243.84 27.94 0)
-		(effects
-			(font
-				(size 1.27 1.27)
-			)
-			(justify left)
-		)
-	)

Commit message: schematic changes - zero DRC errors but I have things to dicuss, and layout footprint work and rearrangment
Parts:
- C109: footprint Capacitor_SMD:C_0603_1608Metric_Pad1.08x0.95mm_HandSolder -> tp_library:C1608X5R1A106M080AC
- C110, C19, C25: footprint Capacitor_SMD:C_0603_1608Metric_Pad1.08x0.95mm_HandSolder -> tp_library:GRM188C81E475KE11D
- C111, C113, C36, C40, C45, C49, C55, C58: footprint Capacitor_SMD:C_0402_1005Metric_Pad0.74x0.62mm_HandSolder -> tp_library:ul_CL05B104KO5NNNC
- C44, C48, C57: footprint Capacitor_SMD:C_0402_1005Metric_Pad0.74x0.62mm_HandSolder -> tp_library:GRM155R6YA224KE01D
Changed lines of the file:
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@@
 			)
 		)
-		(property "Footprint" "Capacitor_SMD:C_0402_1005Metric_Pad0.74x0.62mm_HandSolder"
+		(property "Footprint" "tp_library:ul_CL05B104KO5NNNC"
 			(at 337.5152 76.2 0)
 			(hide yes)
@@
 			)
 		)
-		(property "Footprint" "Capacitor_SMD:C_0402_1005Metric_Pad0.74x0.62mm_HandSolder"
+		(property "Footprint" "tp_library:ul_CL05B104KO5NNNC"
 			(at 350.2152 35.56 0)
 			(hide yes)
@@
 			)
 		)
-		(property "Footprint" "Capacitor_SMD:C_0402_1005Metric_Pad0.74x0.62mm_HandSolder"
+		(property "Footprint" "tp_library:ul_CL05B104KO5NNNC"
 			(at 255.27 69.5452 0)
 			(hide yes)
@@
 			)
 		)
-		(property "Footprint" "Capacitor_SMD:C_0402_1005Metric_Pad0.74x0.62mm_HandSolder"
+		(property "Footprint" "tp_library:GRM155R6YA224KE01D"
 			(at 190.5 80.9752 0)
 			(hide yes)
@@
 			)
 		)
-		(property "Footprint" "Capacitor_SMD:C_0402_1005Metric_Pad0.74x0.62mm_HandSolder"
+		(property "Footprint" "tp_library:ul_CL05B104KO5NNNC"
 			(at 324.8152 125.73 0)
 			(hide yes)
@@
 			)
 		)
-		(property "Footprint" "Capacitor_SMD:C_0402_1005Metric_Pad0.74x0.62mm_HandSolder"
+		(property "Footprint" "tp_library:ul_CL05B104KO5NNNC"
 			(at 259.08 28.9052 0)
 			(hide yes)
@@
 			)
 		)
-		(property "Footprint" "Capacitor_SMD:C_0603_1608Metric_Pad1.08x0.95mm_HandSolder"
+		(property "Footprint" "tp_library:GRM188C81E475KE11D"
 			(at 31.4452 86.36 0)
 			(hide yes)
@@
 			)
 		)
-		(property "Footprint" "Capacitor_SMD:C_0402_1005Metric_Pad0.74x0.62mm_HandSolder"
+		(property "Footprint" "tp_library:GRM155R6YA224KE01D"
 			(at 194.31 40.3352 0)
 			(hide yes)
@@
 			)
 		)
-		(property "Footprint" "Capacitor_SMD:C_0402_1005Metric_Pad0.74x0.62mm_HandSolder"
+		(property "Footprint" "tp_library:ul_CL05B104KO5NNNC"
 			(at 42.8752 194.31 0)
 			(hide yes)
@@
 			)
 		)
-		(property "Footprint" "Capacitor_SMD:C_0402_1005Metric_Pad0.74x0.62mm_HandSolder"
+		(property "Footprint" "tp_library:ul_CL05B104KO5NNNC"
 			(at 63.1952 199.39 0)
 			(hide yes)
@@
 			)
 		)
-		(property "Footprint" "Capacitor_SMD:C_0603_1608Metric_Pad1.08x0.95mm_HandSolder"
+		(property "Footprint" "tp_library:GRM188C81E475KE11D"
 			(at 44.1452 86.36 0)
 			(hide yes)
@@
 			)
 		)
-		(property "Footprint" "Capacitor_SMD:C_0603_1608Metric_Pad1.08x0.95mm_HandSolder"
+		(property "Footprint" "tp_library:GRM188C81E475KE11D"
 			(at 30.1752 147.32 0)
 			(hide yes)
@@
 			)
 		)
-		(property "Footprint" "Capacitor_SMD:C_0603_1608Metric_Pad1.08x0.95mm_HandSolder"
+		(property "Footprint" "tp_library:C1608X5R1A106M080AC"
 			(at 117.8052 147.32 0)
 			(hide yes)
@@
 			)
 		)
-		(property "Footprint" "Capacitor_SMD:C_0402_1005Metric_Pad0.74x0.62mm_HandSolder"
+		(property "Footprint" "tp_library:ul_CL05B104KO5NNNC"
 			(at 254 119.0752 0)
 			(hide yes)
@@
 			)
 		)
-		(property "Footprint" "Capacitor_SMD:C_0402_1005Metric_Pad0.74x0.62mm_HandSolder"
+		(property "Footprint" "tp_library:GRM155R6YA224KE01D"
 			(at 189.23 130.5052 0)
 			(hide yes)
