File: KiCAD/fpga_interconnect/fpga_interconnect.kicad_sch (KiCad schematic)
At the start: 4 parts, among them J1 VGA, J2 Pmod 1, J3 Pmod 2, J4 Conn_02x06_Counter_Clockwise

Commit message: name changes cuz i like lowercase
Parts:
- removed J1: VGA, footprints:AHDF15AKGTAXB, symbol CONN_AHDF15A-KG-TAXB_ASM:AHDF15A-KG-TAXB
- added J1: AHDF15A-KG-TAXB, tp_library:AHDF15AKGTAXB, symbol tp_library:AHDF15A-KG-TAXB
Connections:
- net DATAEN_CMD: now also J1.12
- net GND: now also J1.15
- net HSYNC: now also J1.11
- net IIC1_SCL: now also J1.13
- net IIC1_SDA: now also J1.14
- net PCLK: now also J1.9
- net PDATA0: now also J1.1
- net PDATA1: now also J1.2
- net PDATA2: now also J1.3
- net PDATA3: now also J1.4
- net PDATA4: now also J1.5
- net PDATA5: now also J1.6
- net PDATA6: now also J1.7
- net PDATA7: now also J1.8
- net VSYNC: now also J1.10
Other:
- moved on the sheet: J4

Commit message: fun changes
Parts:
- removed J2: Pmod 1, horizontalHeader:HDRRA12W63P254_2X6_1514X280X635P, symbol 2x6horizontalHeaders:825457-6
- removed J3: Pmod 2, horizontalHeader:HDRRA12W63P254_2X6_1514X280X635P, symbol 2x6horizontalHeaders:825457-6
- added J2, J3: Pmod 2, tp_library:HDRRA12W63P254_2X6_1514X280X635P, symbol tp_library:825457-6
Connections:
- net DATAEN_CMD: now also J3.5
- net GND: now also J2.3, J2.4, J3.3, J3.4, J3.8, J3.9
- net HSYNC: now also J3.6
- net IIC1_SCL: now also J3.7
- net IIC1_SDA: now also J3.10
- net PCLK: now also J3.12
- net PDATA0: now also J2.9
- net PDATA1: now also J2.10
- net PDATA2: now also J2.8
- net PDATA3: now also J2.5
- net PDATA4: now also J2.6
- net PDATA5: now also J2.11
- net PDATA6: now also J2.12
- net PDATA7: now also J2.7
- net VSYNC: now also J3.11
