File: KiCAD/uvBoardV1/uvBoardV1.kicad_pcb (KiCad board)
At the start: 2 copper layers, 15.2 x 17.3 mm, 5 parts, among them J1 Conn_01x03_Pin

Commit message: some doofus goofus
Parts:
- added G***: LOGO, LOGO, B.Cu at (152.3, 66.8)

Commit message: uv board productino files
Other:
- board size 15.2 x 17.3 mm -> 16.2 x 17.8 mm
Changed lines of the file:
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@@
+			)
+		)
+		(property "Digkey Part Number" "1214-SST-10-UV-A130-G405-00CT-ND"
+			(at 0 0 270)
+			(unlocked yes)
+			(layer "F.Fab")
+			(hide yes)
+			(effects
+				(font
+					(size 1 1)
+					(thickness 0.15)
+				)
 			)
 		)
@@
 			)
 		)
+		(property "Digkey Part Number" "XPEBPR-L1-0000-00C01CT-ND "
+			(at 0 0 90)
+			(unlocked yes)
+			(layer "F.Fab")
+			(hide yes)
+			(effects
+				(font
+					(size 1 1)
+					(thickness 0.15)
+				)
+			)
+		)
 		(sheetname "/")
 		(sheetfile "uvBoardV1.kicad_sch")
@@
 			)
 		)
+		(property "Digkey Part Number" "XPEBPR-L1-0000-00C01CT-ND "
+			(at 0 0 270)
+			(unlocked yes)
+			(layer "F.Fab")
+			(hide yes)
+			(effects
+				(font
+					(size 1 1)
+					(thickness 0.15)
+				)
+			)
+		)
 		(sheetname "/")
 		(sheetfile "uvBoardV1.kicad_sch")
@@
 		)
 		(property "MANUFACTURER" "Luminus"
+			(at 0 0 90)
+			(unlocked yes)
+			(layer "F.Fab")
+			(hide yes)
+			(effects
+				(font
+					(size 1 1)
+					(thickness 0.15)
+				)
+			)
+		)
+		(property "Digkey Part Number" "1214-SST-10-UV-A130-G405-00CT-ND"
 			(at 0 0 90)
 			(unlocked yes)
@@
 			)
 		)
+		(property "Digkey Part Number" ""
+			(at 0 0 270)
+			(unlocked yes)
+			(layer "B.Fab")
+			(hide yes)
+			(effects
+				(font
+					(size 1 1)
+					(thickness 0.15)
+				)
+				(justify mirror)
+			)
+		)
 		(property ki_fp_filters "Connector*:*_1x??_*")
 		(sheetname "/")
@@
 		)
 	)
-	(gr_line
-		(start 157.275 57)
-		(end 157.275 60.975)
+	(gr_arc
+		(start 157.614348 60.584493)
+		(mid 152.109728 74.799723)
+		(end 147.278677 60.341696)
 		(stroke
 			(width 0.05)
@@
 		(layer "Edge.Cuts")
 	)
-	(gr_arc
-		(start 157.275 60.975)
-		(mid 152.121878 74.282514)
-		(end 147.599313 60.747707)
+	(gr_line
+		(start 147.278677 60.341697)
+		(end 147.28 57)
 		(stroke
 			(width 0.05)
@@
 	)
 	(gr_line
-		(start 147.600695 60.749454)
-		(end 147.599361 57)
+		(start 157.614348 60.584495)
+		(end 157.61 57)
 		(stroke
 			(width 0.05)
@@
 	(gr_line
 		(start 157 57)
-		(end 157.275 57)
+		(end 157.61 57)
 		(stroke
 			(width 0.05)
@@
 	)
 	(gr_line
-		(start 147.599365 57)
+		(start 147.28 57)
 		(end 157 57)
 		(stroke
@@
 		(polygon
 			(pts
-				(xy 161 57) (xy 161 75) (xy 143 75) (xy 143 57)
-			)
-		)
+				(xy 161 55.1) (xy 161 75) (xy 143 75) (xy 143 55.1)
+			)
+		)
