File: KiCAD/uvBoardV1/uvBoardV1.kicad_sch (KiCad schematic)
At the start: 5 parts, among them J1 Conn_01x03_Pin

Commit message: uv board productino files
Parts:
- D1, D2: Digkey Part Number (none) -> 1214-SST-10-UV-A130-G405-00CT-ND
- D3, D4: Digkey Part Number (none) -> XPEBPR-L1-0000-00C01CT-ND
Other:
- moved on the sheet: D1, D2
Changed lines of the file:
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@@
 	(text "May want to change to a JST later \ninstead of standard header"
 		(exclude_from_sim no)
-		(at 181.864 74.168 0)
+		(at 184.15 74.422 0)
 		(effects
 			(font
@@
 	)
 	(junction
-		(at 151.13 91.44)
+		(at 140.97 92.71)
 		(diameter 0)
 		(color 0 0 0 0)
 	)
 	(junction
-		(at 154.94 91.44)
+		(at 144.78 92.71)
 		(diameter 0)
 		(color 0 0 0 0)
 	)
 	(junction
-		(at 147.32 91.44)
+		(at 137.16 92.71)
 		(diameter 0)
 		(color 0 0 0 0)
 	)
 	(junction
-		(at 153.67 78.74)
+		(at 143.51 80.01)
 		(diameter 0)
 		(color 0 0 0 0)
@@
 	(wire
 		(pts
-			(xy 142.24 91.44) (xy 147.32 91.44)
+			(xy 132.08 92.71) (xy 137.16 92.71)
 		)
 		(stroke
@@
 	(wire
 		(pts
-			(xy 147.32 78.74) (xy 153.67 78.74)
-		)
-		(stroke
-			(width 0)
-			(type default)
-		)
-	)
-	(wire
-		(pts
-			(xy 153.67 78.74) (xy 160.02 78.74)
+			(xy 137.16 80.01) (xy 143.51 80.01)
+		)
+		(stroke
+			(width 0)
+			(type default)
+		)
+	)
+	(wire
+		(pts
+			(xy 143.51 80.01) (xy 149.86 80.01)
 		)
 		(stroke
@@
 	(wire
 		(pts
-			(xy 151.13 91.44) (xy 154.94 91.44)
+			(xy 140.97 92.71) (xy 144.78 92.71)
 		)
 		(stroke
@@
 	(wire
 		(pts
-			(xy 154.94 91.44) (xy 160.02 91.44)
-		)
-		(stroke
-			(width 0)
-			(type default)
-		)
-	)
-	(wire
-		(pts
-			(xy 147.32 91.44) (xy 151.13 91.44)
-		)
-		(stroke
-			(width 0)
-			(type default)
-		)
-	)
-	(wire
-		(pts
-			(xy 153.67 78.74) (xy 153.67 77.47)
+			(xy 144.78 92.71) (xy 149.86 92.71)
+		)
+		(stroke
+			(width 0)
+			(type default)
+		)
+	)
+	(wire
+		(pts
+			(xy 137.16 92.71) (xy 140.97 92.71)
+		)
+		(stroke
+			(width 0)
+			(type default)
+		)
+	)
+	(wire
+		(pts
+			(xy 143.51 80.01) (xy 143.51 78.74)
 		)
 		(stroke
@@
 	)
 	(label "UV+"
-		(at 153.67 77.47 180)
+		(at 143.51 78.74 180)
 		(effects
 			(font
@@
 	(symbol
 		(lib_id "tp_library:SST-10-UV-A130-G405-00")
-		(at 147.32 86.36 270)
+		(at 137.16 87.63 270)
 		(unit 1)
 		(exclude_from_sim no)
@@
 		(dnp no)
 		(property "Reference" "D2"
-			(at 150.368 82.804 90)
+			(at 140.208 84.074 90)
 			(effects
 				(font
@@
 		)
 		(property "Value" "SST-10-UV-A130-G405-00"
-			(at 152.4 85.6296 90)
+			(at 142.24 86.8996 90)
 			(effects
 				(font
@@
 		)
 		(property "Footprint" "tp_library:LED_SST-10-UV-A130-G405-00"
-			(at 147.32 86.36 0)
+			(at 137.16 87.63 0)
 			(effects
 				(font
@@
 		)
 		(property "Datasheet" ""
-			(at 147.32 86.36 0)
+			(at 137.16 87.63 0)
 			(effects
 				(font
@@
 		)
 		(property "Description" ""
-			(at 147.32 86.36 0)
+			(at 137.16 87.63 0)
 			(effects
 				(font
@@
 		)
 		(property "PARTREV" "05"
-			(at 147.32 86.36 0)
+			(at 137.16 87.63 0)
 			(effects
 				(font
@@
 		)
 		(property "STANDARD" "Manufacturer Recommendations"
-			(at 147.32 86.36 0)
+			(at 137.16 87.63 0)
 			(effects
 				(font
@@
 		)
 		(property "MAXIMUM_PACKAGE_HEIGHT" "2.08mm"
-			(at 147.32 86.36 0)
+			(at 137.16 87.63 0)
 			(effects
 				(font
@@
 		)
 		(property "MANUFACTURER" "Luminus"
-			(at 147.32 86.36 0)
+			(at 137.16 87.63 0)
 			(effects
 				(font
@@
 				)
 				(justify bottom)
+				(hide yes)
+			)
+		)
+		(property "Digkey Part Number" "1214-SST-10-UV-A130-G405-00CT-ND"
+			(at 137.16 87.63 90)
+			(effects
+				(font
+					(size 1.27 1.27)
+				)
 				(hide yes)
 			)
@@
 			)
 		)
+		(property "Digkey Part Number" "XPEBPR-L1-0000-00C01CT-ND "
+			(at 140.97 116.84 0)
+			(effects
+				(font
+					(size 1.27 1.27)
+				)
+				(hide yes)
+			)
+		)
 		(pin "1"
 		)
@@
 			)
 		)
+		(property "Digkey Part Number" ""
+			(at 175.26 86.36 0)
+			(effects
+				(font
+					(size 1.27 1.27)
+				)
+				(hide yes)
+			)
+		)
 		(pin "3"
 		)
@@
 	(symbol
 		(lib_id "power:GND")
-		(at 151.13 91.44 0)
+		(at 140.97 92.71 0)
 		(unit 1)
 		(exclude_from_sim no)
@@
 		(fields_autoplaced yes)
 		(property "Reference" "#PWR02"
-			(at 151.13 97.79 0)
+			(at 140.97 99.06 0)
 			(effects
 				(font
@@
 		)
 		(property "Value" "GND"
-			(at 151.13 96.52 0)
+			(at 140.97 97.79 0)
 			(effects
 				(font
@@
 		)
 		(property "Footprint" ""
-			(at 151.13 91.44 0)
+			(at 140.97 92.71 0)
 			(effects
 				(font
@@
 		)
 		(property "Datasheet" ""
-			(at 151.13 91.44 0)
+			(at 140.97 92.71 0)
 			(effects
 				(font
@@
 		)
 		(property "Description" "Power symbol creates a global label with name \"GND\" , ground"
-			(at 151.13 91.44 0)
+			(at 140.97 92.71 0)
 			(effects
 				(font
@@
 	(symbol
 		(lib_id "tp_library:SST-10-UV-A130-G405-00")
-		(at 160.02 86.36 270)
+		(at 149.86 87.63 270)
 		(unit 1)
 		(exclude_from_sim no)
@@
 		(dnp no)
 		(property "Reference" "D1"
-			(at 164.4015 82.8675 90)
+			(at 154.2415 84.1375 90)
 			(effects
 				(font
@@
 		)
 		(property "Value" "SST-10-UV-A130-G405-00"
-			(at 166.37 84.3597 0)
+			(at 156.21 85.6297 0)
 			(effects
 				(font
@@
 		)
 		(property "Footprint" "tp_library:LED_SST-10-UV-A130-G405-00"
-			(at 160.02 86.36 0)
+			(at 149.86 87.63 0)
 			(effects
 				(font
@@
 		)
 		(property "Datasheet" ""
-			(at 160.02 86.36 0)
+			(at 149.86 87.63 0)
 			(effects
 				(font
@@
 		)
 		(property "Description" ""
-			(at 160.02 86.36 0)
+			(at 149.86 87.63 0)
 			(effects
 				(font
@@
 		)
 		(property "PARTREV" "05"
-			(at 160.02 86.36 0)
+			(at 149.86 87.63 0)
 			(effects
 				(font
@@
 		)
 		(property "STANDARD" "Manufacturer Recommendations"
-			(at 160.02 86.36 0)
+			(at 149.86 87.63 0)
 			(effects
 				(font
@@
 		)
 		(property "MAXIMUM_PACKAGE_HEIGHT" "2.08mm"
-			(at 160.02 86.36 0)
+			(at 149.86 87.63 0)
 			(effects
 				(font
@@
 		)
 		(property "MANUFACTURER" "Luminus"
-			(at 160.02 86.36 0)
+			(at 149.86 87.63 0)
 			(effects
 				(font
@@
 				)
 				(justify bottom)
+				(hide yes)
+			)
+		)
+		(property "Digkey Part Number" "1214-SST-10-UV-A130-G405-00CT-ND"
+			(at 149.86 87.63 90)
+			(effects
+				(font
+					(size 1.27 1.27)
+				)
 				(hide yes)
 			)
@@
 				(hide yes)
 			)
+		)
+		(property "Digkey Part Number" "XPEBPR-L1-0000-00C01CT-ND "
+			(at 140.97 102.87 0)
+			(effects
+				(font
+					(size 1.27 1.27)
+				)
+				(hide yes)
+			)
