File: KiCAD/dmd_interconnect/dmd_interconnect.kicad_sch (KiCad schematic)
At the start: 1 part, among them U1 DLP301S

Commit message: dmd interconnect work 1st pass
Changed lines of the file:
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@@
 	(symbol
 		(lib_id "tp_library:DLP301S")
-		(at 156.21 85.09 0)
+		(at 116.84 90.17 0)
 		(unit 1)
 		(exclude_from_sim no)
@@
 		(fields_autoplaced yes)
 		(property "Reference" "U1"
-			(at 158.3533 135.89 0)
+			(at 118.9833 140.97 0)
 			(effects
 				(font
@@
 		)
 		(property "Value" "DLP301S"
-			(at 158.3533 138.43 0)
+			(at 118.9833 143.51 0)
 			(effects
 				(font
@@
 		)
 		(property "Footprint" "tp_library:LGA99_FQS"
-			(at 155.194 119.253 0)
+			(at 115.824 124.333 0)
 			(effects
 				(font
@@
 		)
 		(property "Datasheet" "https://www.ti.com/product/DLP301S"
-			(at 154.94 121.285 0)
+			(at 115.57 126.365 0)
 			(effects
 				(font
@@
 		)
 		(property "Description" ""
-			(at 156.21 41.91 0)
+			(at 116.84 46.99 0)
 			(effects
 				(font
@@
 			)
 		)
+		(pin "D7"
+		)
+		(pin "H6"
+		)
+		(pin "D4"
+		)
+		(pin "F7"
+		)
+		(pin "F5"
+		)
+		(pin "F6"
+		)
+		(pin "D5"
+		)
+		(pin "F4"
+		)
+		(pin "C6"
+		)
+		(pin "C5"
+		)
+		(pin "G6"
+		)
+		(pin "G5"
+		)
+		(pin "H5"
+		)
+		(pin "H4"
+		)
+		(pin "D6"
+		)
+		(pin "H7"
+		)
+		(pin "F2"
+		)
+		(pin "E2"
+		)
+		(pin "A21"
+		)
+		(pin "C2"
+		)
+		(pin "E6"
+		)
+		(pin "F21"
+		)
+		(pin "G20"
+		)
+		(pin "F19"
+		)
+		(pin "D20"
+		)
+		(pin "D22"
+		)
+		(pin "B20"
+		)
+		(pin "E20"
+		)
+		(pin "D2"
+		)
+		(pin "B7"
+		)
+		(pin "C20"
+		)
+		(pin "A19"
+		)
+		(pin "B5"
+		)
+		(pin "D3"
+		)
+		(pin "D23"
+		)
+		(pin "C21"
+		)
+		(pin "D19"
+		)
+		(pin "B2"
+		)
+		(pin "E5"
+		)
+		(pin "B3"
+		)
+		(pin "A20"
+		)
+		(pin "F3"
+		)
+		(pin "D21"
+		)
 		(pin "F20"
 		)
+		(pin "F23"
+		)
+		(pin "F22"
+		)
+		(pin "G21"
+		)
+		(pin "H22"
+		)
+		(pin "H21"
+		)
+		(pin "H19"
+		)
+		(pin "H20"
+		)
 		(pin "E21"
 		)
-		(pin "F19"
-		)
-		(pin "H19"
+		(pin "B4"
+		)
+		(pin "B22"
+		)
+		(pin "H3"
+		)
+		(pin "G22"
+		)
+		(pin "C23"
+		)
+		(pin "A24"
+		)
+		(pin "C22"
+		)
+		(pin "E4"
+		)
+		(pin "B24"
+		)
+		(pin "C4"
+		)
+		(pin "E19"
+		)
+		(pin "B23"
+		)
+		(pin "G19"
+		)
+		(pin "H2"
+		)
+		(pin "A7"
+		)
+		(pin "G24"
+		)
+		(pin "G4"
+		)
+		(pin "H24"
+		)
+		(pin "A4"
+		)
+		(pin "A2"
+		)
+		(pin "C19"
 		)
 		(pin "C7"
 		)
-		(pin "F22"
-		)
-		(pin "G20"
-		)
-		(pin "C22"
-		)
-		(pin "H22"
-		)
-		(pin "A24"
-		)
-		(pin "A7"
-		)
-		(pin "F21"
-		)
-		(pin "B24"
-		)
-		(pin "H20"
-		)
-		(pin "B23"
-		)
-		(pin "D21"
-		)
-		(pin "G21"
-		)
-		(pin "E20"
-		)
-		(pin "H21"
-		)
-		(pin "A2"
-		)
-		(pin "D22"
-		)
 		(pin "A3"
 		)
-		(pin "A4"
-		)
-		(pin "B4"
-		)
-		(pin "B22"
-		)
-		(pin "C19"
-		)
-		(pin "C4"
+		(pin "E22"
+		)
+		(pin "E7"
+		)
+		(pin "G7"
+		)
+		(pin "H23"
+		)
+		(pin "B19"
+		)
+		(pin "B6"
+		)
+		(pin "G3"
+		)
+		(pin "A22"
 		)
 		(pin "G23"
 		)
-		(pin "G7"
-		)
-		(pin "G22"
+		(pin "A6"
+		)
+		(pin "G2"
 		)
 		(pin "C3"
 		)
-		(pin "H23"
-		)
-		(pin "C23"
-		)
-		(pin "H3"
-		)
-		(pin "E22"
-		)
-		(pin "G24"
-		)
-		(pin "B6"
+		(pin "A5"
+		)
+		(pin "B21"
+		)
+		(pin "E3"
+		)
+		(pin "A23"
 		)
 		(pin "E23"
 		)
-		(pin "H24"
-		)
-		(pin "G19"
-		)
-		(pin "E3"
-		)
-		(pin "G3"
-		)
-		(pin "A22"
-		)
-		(pin "A6"
-		)
-		(pin "B21"
-		)
-		(pin "G2"
-		)
-		(pin "E4"
-		)
-		(pin "E19"
-		)
-		(pin "E7"
-		)
-		(pin "G4"
-		)
-		(pin "H2"
-		)
-		(pin "B19"
-		)
-		(pin "A5"
-		)
-		(pin "A23"
-		)
-		(pin "E5"
-		)
-		(pin "H4"
-		)
-		(pin "F4"
-		)
-		(pin "G6"
-		)
-		(pin "G5"
-		)
-		(pin "H5"
-		)
-		(pin "D7"
-		)
-		(pin "C5"
-		)
-		(pin "D4"
-		)
-		(pin "F5"
-		)
-		(pin "C6"
-		)
-		(pin "D6"
-		)
-		(pin "F7"
-		)
-		(pin "H7"
-		)
-		(pin "D5"
-		)
-		(pin "F6"
-		)
-		(pin "H6"
-		)
-		(pin "E6"
-		)
-		(pin "C21"
-		)
-		(pin "A20"
-		)
-		(pin "B7"
-		)
-		(pin "A21"
-		)
-		(pin "B2"
-		)
-		(pin "E2"
-		)
-		(pin "F23"
-		)
-		(pin "B20"
-		)
-		(pin "D2"
-		)
-		(pin "F3"
-		)
-		(pin "C20"
-		)
-		(pin "B3"
-		)
-		(pin "A19"
-		)
-		(pin "C2"
-		)
-		(pin "D23"
-		)
-		(pin "D3"
-		)
-		(pin "B5"
-		)
-		(pin "F2"
-		)
-		(pin "D20"
-		)
-		(pin "D19"
-		)
 		(instances
