File: KiCAD/mainboardTEST/DLPA2005_Interface.kicad_sch (KiCad schematic)
At the start: 37 parts, among them J14 Conn_01x04_Pin, U24 DLPA2005ERSLT

Commit message: idk man maybe didn't save before last commit
Parts:
- C27, C29: footprint (none) -> tp_library:ul_CL05B104KO5NNNC
- C4, C5, C6: footprint (none) -> tp_library:ul_C2012X5R1V106M085AC
Changed lines of the file:
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@@
 			)
 		)
-		(property "Footprint" ""
+		(property "Footprint" "tp_library:ul_C2012X5R1V106M085AC"
 			(at 204.47 54.9148 0)
 			(hide yes)
@@
 			)
 		)
-		(property "Footprint" ""
+		(property "Footprint" "tp_library:ul_CL05B104KO5NNNC"
 			(at 143.2052 195.58 0)
 			(hide yes)
@@
 			)
 		)
-		(property "Footprint" ""
+		(property "Footprint" "tp_library:ul_CL05B104KO5NNNC"
 			(at 210.5152 92.71 0)
 			(hide yes)
@@
 			)
 		)
-		(property "Footprint" ""
+		(property "Footprint" "tp_library:ul_C2012X5R1V106M085AC"
 			(at 233.68 112.0648 0)
 			(hide yes)
@@
 			)
 		)
-		(property "Footprint" ""
+		(property "Footprint" "tp_library:ul_C2012X5R1V106M085AC"
 			(at 233.68 96.8248 0)
 			(hide yes)
