File: KiCAD/mainboardTEST/DLPC1438_Interface.kicad_sch (KiCad schematic)
At the start: 95 parts, among them J10 Conn_01x05_Pin, J2 Conn_01x07_Pin, J29 Conn_01x04_Pin, J3 Conn_02x05_Odd_Even, J31 Conn_01x08_Pin, J4 Conn_01x05_Pin, U12 ECS-2520MV-xxx-xx, U13 MX25L3233FM2, U14 SN74AUP1G06DCKR, U16 DLPC1438ZEZ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

Commit message: idk man maybe didn't save before last commit
Parts:
- R155, R158: footprint STA_RMCF0805_STP -> tp_library:RC0402FR-0710KL
- R156, R157: footprint RES_R-070RL_VIS -> tp_library:ERJ-2GE0R00X
Changed lines of the file:
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@@
 			)
 		)
-		(property "Footprint" "RES_R-070RL_VIS"
+		(property "Footprint" "tp_library:ERJ-2GE0R00X"
 			(at 481.33 -11.43 0)
 			(hide yes)
@@
 			)
 		)
-		(property "Footprint" "RES_R-070RL_VIS"
+		(property "Footprint" "tp_library:ERJ-2GE0R00X"
 			(at 481.33 -16.51 0)
 			(hide yes)
@@
 			)
 		)
-		(property "Footprint" "STA_RMCF0805_STP"
+		(property "Footprint" "tp_library:RC0402FR-0710KL"
 			(at 514.35 -20.32 0)
 			(hide yes)
@@
 			)
 		)
-		(property "Footprint" "STA_RMCF0805_STP"
+		(property "Footprint" "tp_library:RC0402FR-0710KL"
 			(at 502.92 -20.32 0)
 			(hide yes)
