File: KiCAD/mainboardTEST/DMD_Interface.kicad_sch (KiCad schematic)
At the start: 20 parts, among them IC3 SN74AUP1G06DCKR, IC4 SN74AUP1G07DCKR, IC5 SN74AUP1G07DCKR, J1 AXT550124, J30 Conn_01x08_Pin

Commit message: idk man maybe didn't save before last commit
Parts:
- C117, C118, C119: footprint Capacitor_SMD:C_0402_1005Metric -> tp_library:ul_CL05B104KO5NNNC
- R15: footprint STA_RMCF0805_STP -> tp_library:RC0402FR-0710KL
Changed lines of the file:
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@@
 			)
 		)
-		(property "Footprint" "Capacitor_SMD:C_0402_1005Metric"
+		(property "Footprint" "tp_library:ul_CL05B104KO5NNNC"
 			(at 54.3052 39.37 0)
 			(hide yes)
@@
 			)
 		)
-		(property "Footprint" "Capacitor_SMD:C_0402_1005Metric"
+		(property "Footprint" "tp_library:ul_CL05B104KO5NNNC"
 			(at 42.8752 39.37 0)
 			(hide yes)
@@
 			)
 		)
-		(property "Footprint" "STA_RMCF0805_STP"
+		(property "Footprint" "tp_library:RC0402FR-0710KL"
 			(at 163.83 72.39 0)
 			(hide yes)
@@
 			)
 		)
-		(property "Footprint" "Capacitor_SMD:C_0402_1005Metric"
+		(property "Footprint" "tp_library:ul_CL05B104KO5NNNC"
 			(at 65.7352 39.37 0)
 			(hide yes)
