File: KiCAD/mainboardTEST/power_input&generation.kicad_sch (KiCad schematic)
At the start: 85 parts, among them IC1 SN74AUP1G06DCKR, J5 EJ508B, SW2 100SP1T1B4M2QE, U1 XAL5030-472MEC, U2 LMR33610BDDAR, U26 TPS54340DDA, U3 LMR33610BDDAR, U39 TPS62260DDCT, U4 LMR33610BDDAR, U6 74AHC1G08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

Commit message: idk man maybe didn't save before last commit
Parts:
- C110, C19, C25, C43, C47, C56: footprint Capacitor_SMD:C_0603_1608Metric_Pad1.08x0.95mm_HandSolder -> tp_library:CL21A475KBQNNNE
- C111, C113, C26, C36, C40, C45, C49, C55, C58: footprint Capacitor_SMD:C_0603_1608Metric_Pad1.08x0.95mm_HandSolder -> tp_library:ul_CL05B104KO5NNNC
Changed lines of the file:
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@@
 			)
 		)
-		(property "Footprint" "Capacitor_SMD:C_0603_1608Metric_Pad1.08x0.95mm_HandSolder"
+		(property "Footprint" "tp_library:ul_CL05B104KO5NNNC"
 			(at 95.25 77.7748 0)
 			(hide yes)
@@
 			)
 		)
-		(property "Footprint" "Capacitor_SMD:C_0603_1608Metric_Pad1.08x0.95mm_HandSolder"
+		(property "Footprint" "tp_library:ul_CL05B104KO5NNNC"
 			(at 337.5152 76.2 0)
 			(hide yes)
@@
 			)
 		)
-		(property "Footprint" "Capacitor_SMD:C_0603_1608Metric_Pad1.08x0.95mm_HandSolder"
+		(property "Footprint" "tp_library:ul_CL05B104KO5NNNC"
 			(at 63.1952 199.39 0)
 			(hide yes)
@@
 			)
 		)
-		(property "Footprint" "Capacitor_SMD:C_0603_1608Metric_Pad1.08x0.95mm_HandSolder"
+		(property "Footprint" "tp_library:ul_CL05B104KO5NNNC"
 			(at 350.2152 35.56 0)
 			(hide yes)
@@
 			)
 		)
-		(property "Footprint" "Capacitor_SMD:C_0603_1608Metric_Pad1.08x0.95mm_HandSolder"
+		(property "Footprint" "tp_library:ul_CL05B104KO5NNNC"
 			(at 255.27 69.5452 0)
 			(hide yes)
@@
 			)
 		)
-		(property "Footprint" "Capacitor_SMD:C_0603_1608Metric_Pad1.08x0.95mm_HandSolder"
+		(property "Footprint" "tp_library:CL21A475KBQNNNE"
 			(at 189.23 119.0752 0)
 			(hide yes)
@@
 			)
 		)
-		(property "Footprint" "Capacitor_SMD:C_0603_1608Metric_Pad1.08x0.95mm_HandSolder"
+		(property "Footprint" "tp_library:CL21A475KBQNNNE"
 			(at 190.5 69.5452 0)
 			(hide yes)
@@
 			)
 		)
-		(property "Footprint" "Capacitor_SMD:C_0603_1608Metric_Pad1.08x0.95mm_HandSolder"
+		(property "Footprint" "tp_library:ul_CL05B104KO5NNNC"
 			(at 324.8152 125.73 0)
 			(hide yes)
@@
 			)
 		)
-		(property "Footprint" "Capacitor_SMD:C_0603_1608Metric_Pad1.08x0.95mm_HandSolder"
+		(property "Footprint" "tp_library:ul_CL05B104KO5NNNC"
 			(at 259.08 28.9052 0)
 			(hide yes)
@@
 			)
 		)
-		(property "Footprint" "Capacitor_SMD:C_0603_1608Metric_Pad1.08x0.95mm_HandSolder"
+		(property "Footprint" "tp_library:CL21A475KBQNNNE"
 			(at 31.4452 86.36 0)
 			(hide yes)
@@
 			)
 		)
-		(property "Footprint" "Capacitor_SMD:C_0603_1608Metric_Pad1.08x0.95mm_HandSolder"
+		(property "Footprint" "tp_library:ul_CL05B104KO5NNNC"
 			(at 42.8752 194.31 0)
 			(hide yes)
@@
 			)
 		)
-		(property "Footprint" "Capacitor_SMD:C_0603_1608Metric_Pad1.08x0.95mm_HandSolder"
+		(property "Footprint" "tp_library:CL21A475KBQNNNE"
 			(at 44.1452 86.36 0)
 			(hide yes)
@@
 			)
 		)
-		(property "Footprint" "Capacitor_SMD:C_0603_1608Metric_Pad1.08x0.95mm_HandSolder"
+		(property "Footprint" "tp_library:CL21A475KBQNNNE"
 			(at 30.1752 147.32 0)
 			(hide yes)
@@
 			)
 		)
-		(property "Footprint" "Capacitor_SMD:C_0603_1608Metric_Pad1.08x0.95mm_HandSolder"
+		(property "Footprint" "tp_library:CL21A475KBQNNNE"
 			(at 194.31 28.9052 0)
 			(hide yes)
@@
 			)
 		)
-		(property "Footprint" "Capacitor_SMD:C_0603_1608Metric_Pad1.08x0.95mm_HandSolder"
+		(property "Footprint" "tp_library:ul_CL05B104KO5NNNC"
 			(at 254 119.0752 0)
 			(hide yes)
